File: kicad/Serrasoid_TRX.kicad_sch (KiCad schematic)
At the start: 240 parts, among them J1 DC 13.8V, J2 I2C, J3 TJC, J4 ENC, J5 ANT, J6 TX LED, J7 MIC, J8 VOL, J9 SP, K1 G5V-2 DC12, Q1 2SC1815, Q2 2SA1015, Q3 2N7000, Q4 2N3866, Q5 RD06HHF1, Q6 RD16HHF1, Q7 2N3819, Q8 2SC1815, T1 BN43-202 2T:4T, U1 R-78E5.0-1.0, U10 74AC86, U11 74AC86, U12 MCP6004, U13 SA612AN, U14 MC3361, U15 LM386N-1, U16 78L05, U17 MCP6002, U2 L7808, U3 L7805, U4 LP2950-3.3, U5 XIAO ESP32C3, U6 AE-Si5351A, U7 74HCT4017, U8 TLV3501AID, U9 74HC123, X1 10.245MHz, X2 CDBM455C24

Commit message: 回路図を 1 枚（A0）で線による結線に作り直し、表面実装部品をなくす
- ブロックごとに枠で囲み、ブロック内・ブロック間とも線で結線（電源は電源記号）
- コンパレータを TLV3501（SOIC）から MAX913CPA（DIP-8）へ、SHDN はんだジャンパをジャンパピンに
- ERC 違反なし、circuit.py との接続照合 640 ピン一致（tools/verify_sch.py）
- 基板生成スクリプト（配線長を短くする配置 place.py、Freerouting 用 route.sh）を追加。基板は未完成

Co-Authored-By: Claude Opus 5.5 <noreply@anthropic.com>
Parts:
- removed J9: SP, Connector_PinHeader_2.54mm:PinHeader_1x02_P2.54mm_Vertical, symbol Connector_Generic:Conn_01x02
- removed JP1: SHDN, Jumper:SolderJumper-3_P1.3mm_Bridged12_RoundedPad1.0x1.5mm, symbol Jumper:SolderJumper_3_Bridged12
- removed U8: TLV3501AID, Package_SO:SOIC-8_3.9x4.9mm_P1.27mm, symbol Comparator:TLV3501AID
- added J10: SP, Connector_PinHeader_2.54mm:PinHeader_1x02_P2.54mm_Vertical, symbol Connector_Generic:Conn_01x02
- added J9: VOL, Connector_PinHeader_2.54mm:PinHeader_1x03_P2.54mm_Vertical, symbol Connector_Generic:Conn_01x03
- added U8: MAX913CPA, Package_DIP:DIP-8_W7.62mm_Socket, symbol Comparator:LT1016
- J7: value MIC -> LATCH
- J8: value VOL -> MIC
Connections:
- net +5VT: now also J7.3 (Pin_3), U8.1 (V+)
- net GND: now also J7.1 (Pin_1), J10.2 (Pin_2), J9.3 (Pin_3), U8.4 (V-), U8.6 (GND); no longer J7.3 (Pin_3)
- net AF_BYP: no longer names the net of C82.1, U15.7 (BYPASS)
- net AF_DE: no longer names the net of C80.1, C81.1, R57.2
- net AF_DEM: no longer names the net of C90.1, R57.1, U14.9 (AUDIO)
- net AF_IN: no longer names the net of Q8.2 (C), R58.2, U15.3 (+)
- net AF_OUT: no longer names the net of C86.1, R61.1, U15.5
- net ANT: no longer names the net of J5.1 (Pin_1), K1.4
- net CEN_W: no longer names the net of C39.1, R34.1, VR5.2
- net CLIP: no longer names the net of D6.2 (A), D7.1 (K), R30.2, R31.1
- net CLK0: no longer names the net of R11.1, U6.5 (CLK0)
- net CLK0_IN: no longer names the net of R11.2, U7.14 (CLK)
- net CLK1: no longer names the net of R54.1, U6.6 (CLK1)
- net COMP_OUT: no longer names the net of U9.2 (B)
- net COMP_OUT: now also U8.7 (Q)
- net DCDC_IN: no longer names the net of C3.1, L1.2, U1.1 (IN)
- net DEC1: no longer names the net of C77.1, U14.6 (DEC1)
- net DEC2: no longer names the net of C78.1, U14.7 (DEC2)
- net DEV_IN: no longer names the net of C38.2, VR4.1
- net DEV_W: no longer names the net of R33.1, VR4.2
- net DLY1: no longer names the net of C23.1, R16.2, U10.2
- net DLY2: no longer names the net of C24.1, R17.2, U10.5
- net DLY3: no longer names the net of C25.1, R18.2, U10.10
- net DLY4: no longer names the net of C26.1, R19.2, U10.13
- net DLY5: no longer names the net of C27.1, R20.2, U11.2
- net DRV_BN: no longer names the net of R41.2, VR6.1
- net DRV_BW: no longer names the net of C49.1, R42.1, VR6.2
- net DRV_D: no longer names the net of C51.1, L5.2, Q5.3 (D)
- net DRV_G: no longer names the net of Q5.1 (G), R39.2
- net DRV_IN: no longer names the net of C47.2, R39.1, R40.1, R42.2
- net DRV_SW: no longer names the net of C48.1, R40.2
- net ENC_A: no longer names the net of J4.1 (Pin_1), R3.2, U5.4 (D3/A3)
- net ENC_B: no longer names the net of J4.2 (Pin_2), R4.2, U5.1 (D0/A0)
- net ENC_SW: no longer names the net of J4.3 (Pin_3), R5.2, U5.12 (D9/MISO)
- net FD1: no longer names the net of C62.2, C63.1, D8.2 (A), R48.1
- net FD2: no longer names the net of C64.1, D8.1 (K), R49.1, R50.1
- net FWD_ADC: no longer names the net of C65.1, R50.2, U5.2 (D1/A1)
- net IF1: no longer names the net of FL1.3 (OUT), U14.16 (MIX_IN)
- net LIM_IN: no longer names the net of FL2.3 (OUT), U14.5 (LIM_IN)
- net LO_DIV: no longer names the net of C74.1, R54.2, R55.1
- net LO_IN: no longer names the net of C74.2, U13.6 (OSC_B)
- net LPF2: no longer names the net of C59.1, L7.2, L8.1
- net LPF3: no longer names the net of C60.1, L8.2, L9.1
- net LPF_IN: no longer names the net of C58.1, L7.1, T1.3 (SA)
- net MA_IN: no longer names the net of C33.2, R26.1
- net MA_N: no longer names the net of C34.1, R26.2, R27.1, U12.2 (-)
- net MA_OUT: no longer names the net of C34.2, C35.1, R27.2, U12.1
- net MB_N: no longer names the net of R28.1, R29.1, U12.6 (-)
- net MB_OUT: no longer names the net of R28.2, R30.1, U12.7
- net MG_IN: no longer names the net of C35.2, VR3.1
- net MG_W: no longer names the net of U12.5 (+), VR3.2
- net MIC: no longer names the net of C33.1, R25.2
- net MIC: now also J8.1 (Pin_1); no longer J7.1 (Pin_1)
- net MICB: no longer names the net of C32.1, R24.2, R25.1
- net MIC_PTT: no longer names the net of J7.2 (Pin_2)
- net MIC_PTT: now also U8.5 (LATCH); no longer R7.1
- net MIX3: no longer names the net of FL2.1 (IN), U14.3 (MIX_OUT)
- net MIX_IN: no longer names the net of C71.2, U13.1 (IN_A)
- net MIX_INB: no longer names the net of C72.1, U13.2 (IN_B)
- net MIX_OUT: no longer names the net of FL1.1 (IN), U13.4 (OUT_A)
- net MUTE: no longer names the net of R59.1, U5.14 (D7/RX)
- net MUTE_B: no longer names the net of Q8.3 (B), R59.2, R60.1
- net NOISE_ADC: no longer names the net of R67.2, R68.1, U5.3 (D2/A2)
- net NOISE_V: no longer names the net of C93.1, D12.1 (K), R66.1, R67.1
- net NQ_B: no longer names the net of U17.6 (-), U17.7
- net NQ_IN: no longer names the net of C90.2, R64.1
- net NQ_N: no longer names the net of R64.2, R65.1, U17.2 (-)
- net NQ_OUT: no longer names the net of C92.1, R65.2, U17.1
- net NR1: no longer names the net of C92.2, D11.1 (K), D12.2 (A)
- net NREF: no longer names the net of C89.1, R62.2, R63.1, U17.3 (+), U17.5 (+)
- net OSC_B: no longer names the net of C75.1, U14.1 (OSC_B), X1.1
- net OSC_E: no longer names the net of C75.2, C76.1, U14.2 (OSC_E)
- net OS_C: no longer names the net of C21.1, U9.14 (Cext)
- net OS_R: no longer names the net of R15.2, VR2.1
- net OS_RC: no longer names the net of C21.2, U9.15 (RCext), VR2.2, VR2.3
- net PA_BN: no longer names the net of R46.2, VR7.1
- net PA_BW: no longer names the net of C53.1, R47.1, VR7.2
- net PA_D: no longer names the net of C57.1, L6.2, Q6.3 (D)
- net PA_G: no longer names the net of Q6.1 (G), R43.2
- net PA_IN: no longer names the net of C51.2, R43.1, R44.1, R45.1, R47.2
- net PA_SW: no longer names the net of C52.1, R44.2, R45.2
- net PM_OUT: no longer names the net of R16.1, TP3.1, U10.1, U9.13 (Q)
- net PTT_IN: no longer names the net of C14.1, R6.2, R7.2, U5.13 (D8/SCK)
- net QUAD: no longer names the net of R56.1, U14.8 (QUAD), X2.1
- net Q_BUF_B: no longer names the net of C44.2, Q4.2 (B), R35.2, R36.1
- net Q_BUF_C: no longer names the net of C47.1, L4.2, Q4.3 (C)
- net Q_BUF_E: no longer names the net of Q4.1 (E), R37.1
- net Q_BUF_E2: no longer names the net of C45.1, R37.2, R38.1
- net RAMP: no longer names the net of C19.1, Q2.2 (C), Q3.3 (D), TP1.1
- net RAMP: now also U8.2 (+)
- net RAMP_B: no longer names the net of C18.2, D5.1 (K), Q2.3 (B), R13.1
- net RAMP_E: no longer names the net of Q2.1 (E), VR1.2, VR1.3
- net RB1: no longer names the net of C66.1, C67.1, L10.1, TC3.1
- net RB2: no longer names the net of C67.2, C68.1, L11.1, Q7.2 (G), R51.1, TC4.1
- net RE_N: no longer names the net of R12.2, VR1.1
- net RFA_D: no longer names the net of C71.1, Q7.1 (D), R53.2
- net RFA_S: no longer names the net of C69.1, Q7.3 (S), R52.1
- net RLY_B: no longer names the net of Q1.3 (B), R8.2, R9.1
- net RLY_C: no longer names the net of D3.2 (A), K1.16, Q1.2 (C)
- net RST_G: no longer names the net of Q3.2 (G), R14.2
- net RST_P: no longer names the net of R14.1, U7.3 (Q0)
- net RX_ANT: no longer names the net of D10.1 (K), D9.2 (A), K1.6, L10.2 (TAP)
- net SCL: no longer names the net of J2.2 (Pin_2), R2.2, U5.6 (D5/SCL), U6.2 (SCL)
- net SDA: no longer names the net of J2.3 (Pin_3), R1.2, U5.5 (D4/SDA), U6.3 (SDA)
- net SK1: no longer names the net of C36.1, R31.2, R32.1
- net SK2: no longer names the net of C37.1, R32.2, U12.10 (+)
- net SK_OUT: no longer names the net of C36.2, C38.1, U12.8, U12.9 (-)
- net SPK: no longer names the net of C86.2
- net SPK: now also J10.1 (Pin_1)
- net T1_P: no longer names the net of C57.2, T1.1 (AA)
- net TB1: no longer names the net of C41.1, C42.1, L2.1, TC1.1
- net TB2: no longer names the net of C42.2, C43.1, L3.1, TC2.1
- net THRESH: no longer names the net of TP2.1, U12.13 (-), U12.14
- net THRESH: now also U8.3 (-)
- net TH_SUM: no longer names the net of R33.2, R34.2, U12.12 (+)
- net TXBPF_IN: no longer names the net of C30.2, L2.2 (TAP)
- net TXBPF_OUT: no longer names the net of C44.1, L3.2 (TAP)
- net TXDRV: no longer names the net of C30.1, R21.2
- net TXLED: no longer names the net of J6.1 (Pin_1), R10.2
- net TX_EN: no longer names the net of R8.1, U5.11 (D10/MOSI)
- net TX_OUT: no longer names the net of C61.1, C62.1, K1.8, L9.2
- net UART_TX: no longer names the net of J3.2 (Pin_2), U5.7 (D6/TX)
- net VB1: no longer names the net of D4.1 (K), D5.2 (A)
- net VOL_H: no longer names the net of C81.2
- net VOL_H: now also J9.1 (Pin_1); no longer J8.1 (Pin_1)
- net VOL_W: no longer names the net of R58.1
- net VOL_W: now also J9.2 (Pin_2); no longer J8.2 (Pin_2)
- net VREF: no longer names the net of C31.1, C37.2, D6.1 (K), D7.2 (A), R22.2, R23.1, R29.2, U12.3 (+), VR3.3, VR4.3
- net X16: no longer names the net of R20.1, U10.11, U11.1
- net X2: no longer names the net of R17.1, U10.3, U10.4
- net X32: no longer names the net of U11.3, U11.4
- net X32B: no longer names the net of R21.1, TP4.1, U11.6
- net X4: no longer names the net of R18.1, U10.6, U10.9
- net X8: no longer names the net of R19.1, U10.12, U10.8
- net XIAO_5V: no longer names the net of D2.1 (K), U5.8 (VIN)
- net ZOBEL: no longer names the net of C85.1, R61.2
- new net: J8.2 (Pin_2), R7.1
- no-connect marks 31 -> 30
Other:
- note added: "送信: マイク → 送信音声 → セラゾイド変調（915.625kHz で PM）→ 逓倍 ×32 → 送信RF（10W）→ ANT 受信: ANT → 受信（2N3819 → SA612 → 10.7MHz → MC3361 → LM386）→ SP 制御: XIAO ESP32C3 ＋ Si5351（CLK0 = 変調基準 9.15625MHz、CLK1 = 受信局発 18.6MHz） ブロックの中もブロックの間も線で結線（電源・GND は電源記号）"

Commit message: 回路図の論理チェック（第 1 回）: 9 件修正
- リレー駆動のベース抵抗 4.7k → 1k、MAX913 の LE を GND 固定（ジャンパ廃止）
- ワンショットを 74HCT123 に（MAX913 の TTL 出力を受ける）
- 逓倍の遅延を入力周期の 1/4 に直し、RC の後に 74AC14 で整形
- 2N3866 のバイアスを 560/120Ω、出力トランスを 2T:5T（約 8Ω）
- 2N3819 のドレインをチョーク給電、MC3361 周辺をデータシートの試験回路どおりに
- 結果と実物で確認が必要な項目を docs/回路図論理チェック.md に記載

Co-Authored-By: Claude Opus 5.5 <noreply@anthropic.com>
Parts:
- removed J10: SP, Connector_PinHeader_2.54mm:PinHeader_1x02_P2.54mm_Vertical, symbol Connector_Generic:Conn_01x02
- removed unit 2 of U17
- removed unit 3 of U17
- added C94: 0.47u, Capacitor_THT:C_Disc_D5.0mm_W2.5mm_P2.50mm, symbol Device:C
- added L12: 10uH, Inductor_THT:L_Axial_L9.5mm_D4.0mm_P2.54mm_Vertical_Fastron_SMCC, symbol Device:L
- added unit 7 of U10
- added unit 6 of U10
- added unit 3 of U13
- added unit 2 of U13
- added unit 4 of U13
- added unit 5 of U13
- added U18: MCP6002, Package_DIP:DIP-8_W7.62mm_Socket, symbol Amplifier_Operational:MCP6002-xP
- C26: value 47p -> 82p
- C30, C51, C55, C74: value 0.01u -> 0.1u
- C31: value 10u -> 0.01u; footprint Capacitor_THT:CP_Radial_D5.0mm_P2.00mm -> Capacitor_THT:C_Disc_D5.0mm_W2.5mm_P2.50mm; symbol Device:C_Polarized -> Device:C
- C32: value 47u -> 10u
- C33: value 1u -> 47u; footprint Capacitor_THT:C_Disc_D5.0mm_W2.5mm_P2.50mm -> Capacitor_THT:CP_Radial_D5.0mm_P2.00mm; symbol Device:C -> Device:C_Polarized
- C34: value 220p -> 1u; footprint Capacitor_THT:C_Disc_D3.0mm_W1.6mm_P2.50mm -> Capacitor_THT:C_Disc_D5.0mm_W2.5mm_P2.50mm
- C35: value 1u -> 220p; footprint Capacitor_THT:C_Disc_D5.0mm_W2.5mm_P2.50mm -> Capacitor_THT:C_Disc_D3.0mm_W1.6mm_P2.50mm
- C36: value 4.7n -> 1u
- C37: value 2.2n -> 4.7n
- C38: value 1u -> 2.2n
- C39, C82: value 10u -> 1u; footprint Capacitor_THT:CP_Radial_D5.0mm_P2.00mm -> Capacitor_THT:C_Disc_D5.0mm_W2.5mm_P2.50mm; symbol Device:C_Polarized -> Device:C
- C40, C83: value 0.1u -> 10u; footprint Capacitor_THT:C_Disc_D5.0mm_W2.5mm_P2.50mm -> Capacitor_THT:CP_Radial_D5.0mm_P2.00mm; symbol Device:C -> Device:C_Polarized
- C41, C66: value 22p -> 0.1u; footprint Capacitor_THT:C_Disc_D3.0mm_W1.6mm_P2.50mm -> Capacitor_THT:C_Disc_D5.0mm_W2.5mm_P2.50mm
- C42, C67: value 2p -> 22p
- C43, C68: value 22p -> 2p
- C44, C69: value 0.01u -> 22p; footprint Capacitor_THT:C_Disc_D5.0mm_W2.5mm_P2.50mm -> Capacitor_THT:C_Disc_D3.0mm_W1.6mm_P2.50mm
- C50, C54, C65, C73: value 0.1u -> 0.01u
- C56: value 220u -> 0.01u; footprint Capacitor_THT:CP_Radial_D8.0mm_P3.50mm -> Capacitor_THT:C_Disc_D5.0mm_W2.5mm_P2.50mm; symbol Device:C_Polarized -> Device:C
- C57: value 0.1u -> 220u; footprint Capacitor_THT:C_Disc_D5.0mm_W2.5mm_P2.50mm -> Capacitor_THT:CP_Radial_D8.0mm_P3.50mm; symbol Device:C -> Device:C_Polarized
- C58: value 120p -> 0.1u; footprint Capacitor_THT:C_Disc_D5.0mm_W2.5mm_P5.00mm -> Capacitor_THT:C_Disc_D5.0mm_W2.5mm_P2.50mm
- C59: value 220p -> 120p
- C61: value 120p -> 220p
- C62: value 4.7p -> 120p; footprint Capacitor_THT:C_Disc_D3.0mm_W1.6mm_P2.50mm -> Capacitor_THT:C_Disc_D5.0mm_W2.5mm_P5.00mm
- C63: value 100p -> 4.7p
- C64: value 0.01u -> 100p; footprint Capacitor_THT:C_Disc_D5.0mm_W2.5mm_P2.50mm -> Capacitor_THT:C_Disc_D3.0mm_W1.6mm_P2.50mm
- C75: value 68p -> 0.01u; footprint Capacitor_THT:C_Disc_D3.0mm_W1.6mm_P2.50mm -> Capacitor_THT:C_Disc_D5.0mm_W2.5mm_P2.50mm
- C76: value 220p -> 68p
- C77: value 0.1u -> 220p; footprint Capacitor_THT:C_Disc_D5.0mm_W2.5mm_P2.50mm -> Capacitor_THT:C_Disc_D3.0mm_W1.6mm_P2.50mm
- C80: value 0.047u -> 0.1u
- C81: value 1u -> 0.047u
- C84: value 100u -> 0.1u; footprint Capacitor_THT:CP_Radial_D6.3mm_P2.50mm -> Capacitor_THT:C_Disc_D5.0mm_W2.5mm_P2.50mm; symbol Device:C_Polarized -> Device:C
- C85: value 0.047u -> 100u; footprint Capacitor_THT:C_Disc_D5.0mm_W2.5mm_P2.50mm -> Capacitor_THT:CP_Radial_D6.3mm_P2.50mm; symbol Device:C -> Device:C_Polarized
- C86: value 220u -> 0.047u; footprint Capacitor_THT:CP_Radial_D6.3mm_P2.50mm -> Capacitor_THT:C_Disc_D5.0mm_W2.5mm_P2.50mm; symbol Device:C_Polarized -> Device:C
- C87: value 0.1u -> 220u; footprint Capacitor_THT:C_Disc_D5.0mm_W2.5mm_P2.50mm -> Capacitor_THT:CP_Radial_D6.3mm_P2.50mm; symbol Device:C -> Device:C_Polarized
- C88: value 10u -> 0.1u; footprint Capacitor_THT:CP_Radial_D5.0mm_P2.00mm -> Capacitor_THT:C_Disc_D5.0mm_W2.5mm_P2.50mm; symbol Device:C_Polarized -> Device:C
- C90: value 2.2n -> 10u; footprint Capacitor_THT:C_Disc_D5.0mm_W2.5mm_P2.50mm -> Capacitor_THT:CP_Radial_D5.0mm_P2.00mm; symbol Device:C -> Device:C_Polarized
- C91: value 0.1u -> 2.2n
- C93: value 0.47u -> 0.1u
- J7: value LATCH -> MIC
- J8: value MIC -> VOL
- J9: value VOL -> SP; footprint Connector_PinHeader_2.54mm:PinHeader_1x03_P2.54mm_Vertical -> Connector_PinHeader_2.54mm:PinHeader_1x02_P2.54mm_Vertical; symbol Connector_Generic:Conn_01x03 -> Connector_Generic:Conn_01x02
- R16: value 2k -> 3.9k
- R17: value 1k -> 1.8k
- R18: value 510 -> 910
- R20: value 270 -> 330
- R35: value 4.7k -> 560
- R36: value 1k -> 120
- R56: value 6.8k -> 20k
- R8: value 4.7k -> 1k
- T1: value BN43-202 2T:4T -> BN43-202 2T:5T
- U10: value 74AC86 -> 74AC14; symbol 74xx:74HC86 -> 74xx:74HC14
- U12: value MCP6004 -> 74AC86; symbol Amplifier_Operational:MCP6004 -> 74xx:74HC86
- U13: value SA612AN -> MCP6004; footprint Package_DIP:DIP-8_W7.62mm_Socket -> Package_DIP:DIP-14_W7.62mm_Socket; symbol Serrasoid_TRX:SA612 -> Amplifier_Operational:MCP6004
- U14: value MC3361 -> SA612AN; footprint Package_DIP:DIP-16_W7.62mm_Socket -> Package_DIP:DIP-8_W7.62mm_Socket; symbol Serrasoid_TRX:MC3361 -> Serrasoid_TRX:SA612
- U15: value LM386N-1 -> MC3361; footprint Package_DIP:DIP-8_W7.62mm_Socket -> Package_DIP:DIP-16_W7.62mm_Socket; symbol Amplifier_Audio:LM386 -> Serrasoid_TRX:MC3361
- U16: value 78L05 -> LM386N-1; footprint Package_TO_SOT_THT:TO-92_Inline -> Package_DIP:DIP-8_W7.62mm_Socket; symbol Regulator_Linear:L78L05_TO92 -> Amplifier_Audio:LM386
- U17: value MCP6002 -> 78L05; footprint Package_DIP:DIP-8_W7.62mm_Socket -> Package_TO_SOT_THT:TO-92_Inline; symbol Amplifier_Operational:MCP6002-xP -> Regulator_Linear:L78L05_TO92
- U9: value 74HC123 -> 74HCT123
Connections:
- net +13V8: now also C51.1, C57.1; no longer C50.1, C54.1
- net +5VA: now also C74.1, C77.2, C78.2, C79.2, C80.1, C89.1, C92.1, U14.8 (VCC), U15.4 (VCC), U17.1 (VO), X1.2, U18.8 (V+); no longer C73.1, C79.1, C88.1, C91.1, U13.8 (VCC), U14.4 (VCC), U16.1 (VO)
- net +5VT: now also C30.1, C41.1, U12.14 (VCC), U10.14 (VCC), U13.4 (V+); no longer C40.1, J7.3 (Pin_3), U10.14 (VCC), U12.4 (V+)
- net GND: now also C30.2, C33.2, C42.2, C44.2, C47.2, C51.2, C57.2, C62.2, C67.2, C71.2, C74.2, C81.2, C86.2, C90.2, C92.2, J7.3 (Pin_3), J9.2 (Pin_2), U12.10, U12.12, U12.13, U12.5, U12.7 (GND), U12.9, U14.3 (GND), U15.15 (GND), U16.4 (GND), U17.2 (GND), U8.5 (LATCH), C94.2, U10.13, U10.7 (GND), U13.11 (V-), U18.4 (V-); no longer C31.2, C39.2, C43.2, C45.2, C48.2, C52.2, C58.2, C63.2, C68.2, C72.2, C76.2, C77.2, C78.2, C79.2, C82.2, C87.2, C91.2, C93.2, J7.1 (Pin_1), J9.3 (Pin_3), U10.7 (GND), U11.10, U11.12, U11.13, U11.5, U11.9, U12.11 (V-), U13.3 (GND), U14.15 (GND), U15.2 (-), U15.4 (GND), X1.2
- net RX8V: now also C71.1, C85.1, C88.1, U16.6 (V+), U17.3 (VI), L12.1; no longer C70.1, C83.1, C87.1, U15.6 (V+), U16.3 (VI)
- net TX8V: now also C47.1; no longer C46.1
- net at R21.1, TP4.1: now also U12.6; no longer U11.6
- net at D6.1 (K), D7.2 (A), R22.2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: now also C32.1, C38.2, U13.3 (+); no longer C31.1, C37.2, U12.3 (+)
- net at D12.1 (K), R66.1, R67.1: now also C94.1; no longer C93.1
- net at C78.1: now also U15.6 (DEC1); no longer U14.7 (DEC2)
- net at L4.2, Q4.3 (C): now also C48.1; no longer C47.1
- net at R39.1, R40.1, R42.2: now also C48.2; no longer C47.2
- net at R47.1, VR7.2: now also C54.1; no longer C53.1
- net at VR3.1: now also C36.2; no longer C35.2
- net at VR3.2: now also U13.5 (+); no longer U12.5 (+)
- net at R56.1, X2.1: now also U15.8 (QUAD); no longer U14.8 (QUAD)
- net at D8.1 (K), R49.1, R50.1: now also C65.1; no longer C64.1
- net at D8.2 (A), R48.1: now also C63.2, C64.1; no longer C62.2, C63.1
- net at L7.2, L8.1: now also C60.1; no longer C59.1
- net at L8.2, L9.1: now also C61.1; no longer C60.1
- net at C67.1, L10.1, TC3.1: now also C68.1; no longer C66.1
- net at L11.1, Q7.2 (G), R51.1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: now also C68.2, C69.1; no longer C67.2, C68.1
- net at R26.2, R27.1: now also C35.1, U13.2 (-); no longer C34.1, U12.2 (-)
- net at FL2.1 (IN): now also U15.3 (MIX_OUT); no longer U14.3 (MIX_OUT)
- net at FL2.3 (OUT): now also U15.5 (LIM_IN); no longer U14.5 (LIM_IN)
- net at D11.1 (K), D12.2 (A): now also C93.2; no longer C92.2
- net at R50.2, U5.2 (D1/A1): now also C66.1; no longer C65.1
- net at R28.2, R30.1: now also U13.7; no longer U12.7
- net at C62.1, K1.8, L9.2: now also C63.1; no longer C61.1
- net at L7.1, T1.3 (SA): now also C59.1; no longer C58.1
- net at R61.2: now also C86.1; no longer C85.1
- net at L3.1, TC2.1: now also C43.2, C44.1; no longer C42.2, C43.1
- net at R33.2, R34.2: now also U13.12 (+); no longer U12.12 (+)
- net at TP2.1, U8.3 (-): now also U13.13 (-), U13.14; no longer U12.13 (-), U12.14
- net at R37.2, R38.1: now also C46.1; no longer C45.1
- net at U13.1: now also C35.2, C36.1, R27.2; no longer C71.2
- net at C72.1: now also Q7.1 (D), R53.2, L12.2; no longer U13.2 (IN_B)
- net at FL1.1 (IN): now also U14.4 (OUT_A); no longer U13.4 (OUT_A)
- net at J7.2 (Pin_2): now also R7.1; no longer U8.5 (LATCH)
- net at C25.1, R18.2: now also U10.5; no longer U10.10
- net at R64.1: now also C91.2; no longer C90.2
- net at C81.1, R57.2: now also C82.1; no longer C80.1
- net at J9.1 (Pin_1): now also C87.2; no longer C81.2
- net at L6.2, Q6.3 (D): now also C58.1; no longer C57.1
- net at R24.2, R25.1: now also C33.1; no longer C32.1
- net at T1.1 (AA): now also C58.2; no longer C57.2
- net at R58.1: now also J8.2 (Pin_2); no longer J9.2 (Pin_2)
- net at Q8.2 (C), R58.2: now also U16.3 (+); no longer U15.3 (+)
- net at Q7.3 (S), R52.1: now also C70.1; no longer C69.1
- net at C27.1, R20.2: now also U10.11; no longer U11.2
- net at R16.1, TP3.1, U9.13 (Q): now also U11.1; no longer U10.1
- net at R28.1, R29.1: now also U13.6 (-); no longer U12.6 (-)
- net at FL1.3 (OUT): now also U15.16 (MIX_IN); no longer U14.16 (MIX_IN)
- net at R26.1: now also C34.2; no longer C33.2
- net at R34.1, VR5.2: now also C40.1; no longer C39.1
- net at R31.2, R32.1: now also C37.1; no longer C36.1
- net at R43.1, R44.1, R45.1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: now also C52.2; no longer C51.2
- net at Q4.2 (B), R35.2, R36.1: now also C45.2; no longer C44.2
- net at R62.2, R63.1: now also C90.1, U18.3 (+), U18.5 (+); no longer C89.1, U17.3 (+)
- net at L3.2 (TAP): now also C45.1; no longer C44.1
- net at U11.8: now also R19.1, U11.12
- net at R40.2: now also C49.1; no longer C48.1
- net at C26.1, R19.2: now also U10.9; no longer U10.13
- net at VR4.1: now also C39.2; no longer C38.2
- net at L5.2, Q5.3 (D): now also C52.1; no longer C51.1
- net at C23.1, R16.2: now also U10.1; no longer U10.2
- net at R21.2: now also C31.1; no longer C30.1
- net at L2.2 (TAP): now also C31.2; no longer C30.2
- net at R44.2, R45.2: now also C53.1; no longer C52.1
- net at C42.1, L2.1, TC1.1: now also C43.1; no longer C41.1
- net at R54.2, R55.1: now also C75.1; no longer C74.1
- net at R64.2, R65.1: now also U18.2 (-); no longer U17.2 (-)
- net at U11.11: now also R20.1, U12.1
- net at C24.1, R17.2: now also U10.3; no longer U10.5
- net at R42.1, VR6.2: now also C50.1; no longer C49.1
- net at U15.1 (OSC_B): now also C76.1, X1.1
- net at U15.7 (DEC2): now also C79.1; no longer C82.1
- net at C77.1: now also C76.2, U15.2 (OSC_E); no longer U14.6 (DEC1)
- net at U11.3, U11.4: now also R17.1
- new net: C38.1, R32.2, U13.10 (+)
- new net: C37.2, C39.1, U13.8, U13.9 (-)
- new net: C34.1, J7.1 (Pin_1), R25.2
- new net: U10.6, U11.10
- new net: C91.1, R57.1, U15.9 (AUDIO)
- new net: C83.1, U16.7 (BYPASS)
- new net: C87.1, R61.1, U16.5
- new net: C72.2, U14.1 (IN_A)
- new net: R18.1, U11.6, U11.9
- new net: U10.8, U11.13
- new net: U10.10, U12.2
- new net: U10.2, U11.2
- new net: C73.1, U14.2 (IN_B)
- new net: C75.2, U14.6 (OSC_B)
- new net: U12.3, U12.4
- new net: C82.2, J8.1 (Pin_1)
- new net: C93.1, R65.2, U18.1
- new net: U10.4, U11.5
- new net: U18.6 (-), U18.7
- now unconnected: U12.8
- no-connect marks 30 -> 31
Other:
- moved on the sheet: C17, C18, C19, C20, C21, C22, C23, C24, C25, C26, C27, C28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
