File: kicad/Serrasoid_TRX.kicad_sch (KiCad schematic)
At the start: 242 parts, among them J1 DC 13.8V, J2 I2C, J3 TJC, J4 ENC, J5 ANT, J6 TX LED, J7 MIC, J8 VOL, J9 SP, K1 G5V-2 DC12, Q1 2SC1815, Q2 2SA1015, Q3 2N7000, Q4 2N3866, Q5 RD06HHF1, Q6 RD16HHF1, Q7 2N3819, Q8 2SC1815, T1 BN43-202 2T:5T, U1 R-78E5.0-1.0, U10 74AC14, U11 74AC86, U12 74AC86, U13 MCP6004, U14 SA612AN, U15 MC3361, U16 LM386N-1, U17 78L05, U18 MCP6002, U2 L7808, U3 L7805, U4 LP2950-3.3, U5 XIAO ESP32C3, U6 AE-Si5351A, U7 74HCT4017, U8 MAX913CPA, U9 74HCT123, X1 10.245MHz, X2 CDBM455C24

Commit message: 回路図の論理チェック（第 2 回）: 2 件修正し、基板を作り直す
- XIAO の D0（GPIO2、起動時に High が必要）からエンコーダ B 相を外し、D0 = PTT、D8 = エンコーダ B 相に
- SA612 の局発入力を範囲（200〜300mVp-p）の中央に: R54 1k → 1.2kΩ（約 0.25Vp-p）
- C58 は積層セラミック（約 1.6Arms）と部品表に明記
- PTT・エンコーダ周りの回路図の配置を、ピンの入れ替えに合わせて手で置き直す
- 回路図: ERC 違反なし、接続照合 655 ピン一致。基板: 配置・配線をやり直し DRC エラー 0・未接続 0・食い違い 0
- 結果を docs/回路図論理チェック.md に追記、README の XIAO のピン表を更新

Co-Authored-By: Claude Opus 5.5 <noreply@anthropic.com>
Parts:
- R54: value 1k -> 1.2k
Connections:
- net at J4.2 (Pin_2), R4.2: now also U5.13 (D8/SCK); no longer U5.1 (D0/A0)
- net at C14.1, R6.2, R7.2: now also U5.1 (D0/A0); no longer U5.13 (D8/SCK)
Other:
- moved on the sheet: C14, C67, C68, C69, C70, C71, C72, C73, C74, C75, C76, C77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

Commit message: 部品番号を回路図の位置順に振り直す（PSN_TRX 2026-10-15 と同じ方法）
- 種類ごとに回路図の X の小さい順、同じ X は Y の順（多ユニットは最も小さいユニットの位置）。242 点のうち 206 点が変更
- tools/renumber.py: 回路図・基板の部品番号と、番号から作る UUID、基板のネット名（Net-(C23-Pad1) など 140 個）を書き換え、
  circuit.py の RENUMBER（仮の番号 → 最終の番号）・LAYOUT・注記、資料・ケースの番号も置き換える
- 新旧の対応表 kicad/refdes_map_2026-10-16.csv。チェックの記録（回路図論理チェック・基板チェック）は旧番号のまま注記
- 確認: 回路図と circuit.py の照合 655 ピン一致、ERC 0、DRC エラー 0・未接続 0・回路図との食い違い 0（シルクの警告のみ）、
  LAYOUT と回路図の位置がブロックごとに一致
- 部品表・回路図 PDF・部品実装図・A3 配置図・動作説明 docx を作り直し

Co-Authored-By: Claude Opus 5.5 <noreply@anthropic.com>
Parts:
- removed unit 3 of U10
- removed unit 7 of U10
- removed unit 4 of U10
- removed unit 5 of U10
- removed unit 2 of U10
- removed unit 6 of U10
- removed unit 4 of U12
- removed unit 5 of U12
- removed unit 2 of U12
- removed unit 3 of U12
- removed unit 3 of U13
- removed unit 2 of U13
- removed unit 4 of U13
- removed unit 5 of U13
- removed unit 3 of U18
- removed unit 2 of U18
- removed unit 2 of U9
- removed unit 3 of U9
- added unit 5 of U1
- added unit 6 of U1
- added unit 4 of U1
- added unit 2 of U1
- added unit 3 of U1
- added unit 7 of U1
- added unit 3 of U16
- added unit 2 of U16
- added unit 2 of U17
- added unit 3 of U17
- added unit 2 of U2
- added unit 5 of U2
- added unit 4 of U2
- added unit 3 of U2
- added unit 2 of U8
- added unit 3 of U8
- added unit 5 of U8
- added unit 4 of U8
- C1: value 470u -> 100p; footprint Capacitor_THT:CP_Radial_D8.0mm_P3.50mm -> Capacitor_THT:C_Disc_D3.0mm_W1.6mm_P2.50mm; symbol Device:C_Polarized -> Device:C
- C10, C32: value 10u -> 0.01u; footprint Capacitor_THT:CP_Radial_D5.0mm_P2.00mm -> Capacitor_THT:C_Disc_D5.0mm_W2.5mm_P2.50mm; symbol Device:C_Polarized -> Device:C
- C11, C18, C28, C55, C79: value 0.1u -> 10u; footprint Capacitor_THT:C_Disc_D5.0mm_W2.5mm_P2.50mm -> Capacitor_THT:CP_Radial_D5.0mm_P2.00mm; symbol Device:C -> Device:C_Polarized
- C14, C47, C50, C75: value 0.01u -> 0.1u
- C15, C16: value 47u -> 0.01u; footprint Capacitor_THT:CP_Radial_D5.0mm_P2.00mm -> Capacitor_THT:C_Disc_D5.0mm_W2.5mm_P2.50mm; symbol Device:C_Polarized -> Device:C
- C17, C29: value 0.1u -> 0.01u
- C19, C24, C64: value 100p -> 0.01u; footprint Capacitor_THT:C_Disc_D3.0mm_W1.6mm_P2.50mm -> Capacitor_THT:C_Disc_D5.0mm_W2.5mm_P2.50mm
- C2, C5, C58: value 0.1u -> 22p; footprint Capacitor_THT:C_Disc_D5.0mm_W2.5mm_P2.50mm -> Capacitor_THT:C_Disc_D3.0mm_W1.6mm_P2.50mm
- C21: value 100p -> 10u; footprint Capacitor_THT:C_Disc_D3.0mm_W1.6mm_P2.50mm -> Capacitor_THT:CP_Radial_D5.0mm_P2.00mm; symbol Device:C -> Device:C_Polarized
- C25: value 100p -> 0.1u; footprint Capacitor_THT:C_Disc_D3.0mm_W1.6mm_P2.50mm -> Capacitor_THT:C_Disc_D5.0mm_W2.5mm_P2.50mm
- C26: value 82p -> 0.1u; footprint Capacitor_THT:C_Disc_D3.0mm_W1.6mm_P2.50mm -> Capacitor_THT:C_Disc_D5.0mm_W2.5mm_P2.50mm
- C27: value 47p -> 0.01u; footprint Capacitor_THT:C_Disc_D3.0mm_W1.6mm_P2.50mm -> Capacitor_THT:C_Disc_D5.0mm_W2.5mm_P2.50mm
- C3: value 10u -> 2p; footprint Capacitor_THT:CP_Radial_D5.0mm_P2.00mm -> Capacitor_THT:C_Disc_D3.0mm_W1.6mm_P2.50mm; symbol Device:C_Polarized -> Device:C
- C31: value 0.01u -> 82p; footprint Capacitor_THT:C_Disc_D5.0mm_W2.5mm_P2.50mm -> Capacitor_THT:C_Disc_D3.0mm_W1.6mm_P2.50mm
- C33: value 47u -> 0.1u; footprint Capacitor_THT:CP_Radial_D5.0mm_P2.00mm -> Capacitor_THT:C_Disc_D5.0mm_W2.5mm_P2.50mm; symbol Device:C_Polarized -> Device:C
- C34, C36, C82: value 1u -> 0.1u
- C35: value 220p -> 0.01u; footprint Capacitor_THT:C_Disc_D3.0mm_W1.6mm_P2.50mm -> Capacitor_THT:C_Disc_D5.0mm_W2.5mm_P2.50mm
- C37: value 4.7n -> 220u; footprint Capacitor_THT:C_Disc_D5.0mm_W2.5mm_P2.50mm -> Capacitor_THT:CP_Radial_D8.0mm_P3.50mm; symbol Device:C -> Device:C_Polarized
- C38: value 2.2n -> 120p; footprint Capacitor_THT:C_Disc_D5.0mm_W2.5mm_P2.50mm -> Capacitor_THT:C_Disc_D5.0mm_W2.5mm_P5.00mm
- C39: value 1u -> 0.01u
- C4: value 10u -> 470u; footprint Capacitor_THT:CP_Radial_D5.0mm_P2.00mm -> Capacitor_THT:CP_Radial_D8.0mm_P3.50mm
- C40: value 10u -> 47p; footprint Capacitor_THT:CP_Radial_D5.0mm_P2.00mm -> Capacitor_THT:C_Disc_D3.0mm_W1.6mm_P2.50mm; symbol Device:C_Polarized -> Device:C
- C41: value 0.1u -> 220p; footprint Capacitor_THT:C_Disc_D5.0mm_W2.5mm_P2.50mm -> Capacitor_THT:C_Disc_D5.0mm_W2.5mm_P5.00mm
- C42: value 22p -> 220p; footprint Capacitor_THT:C_Disc_D3.0mm_W1.6mm_P2.50mm -> Capacitor_THT:C_Disc_D5.0mm_W2.5mm_P5.00mm
- C43: value 2p -> 120p; footprint Capacitor_THT:C_Disc_D3.0mm_W1.6mm_P2.50mm -> Capacitor_THT:C_Disc_D5.0mm_W2.5mm_P5.00mm
- C44: value 22p -> 4.7p
- C45, C73: value 0.01u -> 100p; footprint Capacitor_THT:C_Disc_D5.0mm_W2.5mm_P2.50mm -> Capacitor_THT:C_Disc_D3.0mm_W1.6mm_P2.50mm
- C49, C52: value 0.01u -> 47u; footprint Capacitor_THT:C_Disc_D5.0mm_W2.5mm_P2.50mm -> Capacitor_THT:CP_Radial_D5.0mm_P2.00mm; symbol Device:C -> Device:C_Polarized
- C51: value 0.1u -> 47u; footprint Capacitor_THT:C_Disc_D5.0mm_W2.5mm_P2.50mm -> Capacitor_THT:CP_Radial_D5.0mm_P2.00mm; symbol Device:C -> Device:C_Polarized
- C53: value 0.01u -> 22p; footprint Capacitor_THT:C_Disc_D5.0mm_W2.5mm_P2.50mm -> Capacitor_THT:C_Disc_D3.0mm_W1.6mm_P2.50mm
- C54: value 0.01u -> 1u
- C56: value 0.01u -> 2p; footprint Capacitor_THT:C_Disc_D5.0mm_W2.5mm_P2.50mm -> Capacitor_THT:C_Disc_D3.0mm_W1.6mm_P2.50mm
- C57: value 220u -> 10u; footprint Capacitor_THT:CP_Radial_D8.0mm_P3.50mm -> Capacitor_THT:CP_Radial_D5.0mm_P2.00mm
- C59: value 120p -> 220p; footprint Capacitor_THT:C_Disc_D5.0mm_W2.5mm_P5.00mm -> Capacitor_THT:C_Disc_D3.0mm_W1.6mm_P2.50mm
- C60: value 220p -> 1u; footprint Capacitor_THT:C_Disc_D5.0mm_W2.5mm_P5.00mm -> Capacitor_THT:C_Disc_D5.0mm_W2.5mm_P2.50mm
- C61: value 220p -> 0.01u; footprint Capacitor_THT:C_Disc_D5.0mm_W2.5mm_P5.00mm -> Capacitor_THT:C_Disc_D5.0mm_W2.5mm_P2.50mm
- C62: value 120p -> 0.01u; footprint Capacitor_THT:C_Disc_D5.0mm_W2.5mm_P5.00mm -> Capacitor_THT:C_Disc_D5.0mm_W2.5mm_P2.50mm
- C63: value 4.7p -> 0.01u; footprint Capacitor_THT:C_Disc_D3.0mm_W1.6mm_P2.50mm -> Capacitor_THT:C_Disc_D5.0mm_W2.5mm_P2.50mm
- C67, C69: value 22p -> 0.1u; footprint Capacitor_THT:C_Disc_D3.0mm_W1.6mm_P2.50mm -> Capacitor_THT:C_Disc_D5.0mm_W2.5mm_P2.50mm
- C68: value 2p -> 0.1u; footprint Capacitor_THT:C_Disc_D3.0mm_W1.6mm_P2.50mm -> Capacitor_THT:C_Disc_D5.0mm_W2.5mm_P2.50mm
- C7, C90: value 10u -> 0.1u; footprint Capacitor_THT:CP_Radial_D5.0mm_P2.00mm -> Capacitor_THT:C_Disc_D5.0mm_W2.5mm_P2.50mm; symbol Device:C_Polarized -> Device:C
- C70: value 0.01u -> 68p; footprint Capacitor_THT:C_Disc_D5.0mm_W2.5mm_P2.50mm -> Capacitor_THT:C_Disc_D3.0mm_W1.6mm_P2.50mm
- C71: value 0.01u -> 220p; footprint Capacitor_THT:C_Disc_D5.0mm_W2.5mm_P2.50mm -> Capacitor_THT:C_Disc_D3.0mm_W1.6mm_P2.50mm
- C72: value 0.01u -> 2.2n
- C74: value 0.1u -> 4.7n
- C76: value 68p -> 0.1u; footprint Capacitor_THT:C_Disc_D3.0mm_W1.6mm_P2.50mm -> Capacitor_THT:C_Disc_D5.0mm_W2.5mm_P2.50mm
- C77: value 220p -> 1u; footprint Capacitor_THT:C_Disc_D3.0mm_W1.6mm_P2.50mm -> Capacitor_THT:C_Disc_D5.0mm_W2.5mm_P2.50mm
- C78: value 0.1u -> 2.2n
- C80: value 0.1u -> 0.047u
- C81: value 0.047u -> 1u
- C84, C9: value 0.1u -> 100p; footprint Capacitor_THT:C_Disc_D5.0mm_W2.5mm_P2.50mm -> Capacitor_THT:C_Disc_D3.0mm_W1.6mm_P2.50mm
- C85: value 100u -> 0.1u; footprint Capacitor_THT:CP_Radial_D6.3mm_P2.50mm -> Capacitor_THT:C_Disc_D5.0mm_W2.5mm_P2.50mm; symbol Device:C_Polarized -> Device:C
- C86: value 0.047u -> 0.1u
- C87: value 220u -> 100u
- C91: value 2.2n -> 0.047u
- C92: value 0.1u -> 0.47u
- C93: value 0.1u -> 220u; footprint Capacitor_THT:C_Disc_D5.0mm_W2.5mm_P2.50mm -> Capacitor_THT:CP_Radial_D6.3mm_P2.50mm; symbol Device:C -> Device:C_Polarized
- C94: value 0.47u -> 0.1u
- D2: value 1N5819 -> 1N60; footprint Diode_THT:D_DO-41_SOD81_P5.08mm_Vertical_AnodeUp -> Diode_THT:D_DO-35_SOD27_P2.54mm_Vertical_AnodeUp; symbol Diode:1N5819 -> Device:D
- D3: value 1N4001 -> 1N5819; symbol Diode:1N4001 -> Diode:1N5819
- D4: value 1N4148 -> 1N4001; footprint Diode_THT:D_DO-35_SOD27_P2.54mm_Vertical_AnodeUp -> Diode_THT:D_DO-41_SOD81_P5.08mm_Vertical_AnodeUp; symbol Diode:1N4148 -> Diode:1N4001
- D8: value 1N60 -> 1N4148; symbol Device:D -> Diode:1N4148
- J5: value ANT -> MIC; footprint Connector_Wire:SolderWire-1sqmm_1x02_P5.4mm_D1.4mm_OD2.7mm -> Connector_PinHeader_2.54mm:PinHeader_1x03_P2.54mm_Vertical; symbol Connector_Generic:Conn_01x02 -> Connector_Generic:Conn_01x03
- J6: value TX LED -> ANT; footprint Connector_PinHeader_2.54mm:PinHeader_1x02_P2.54mm_Vertical -> Connector_Wire:SolderWire-1sqmm_1x02_P5.4mm_D1.4mm_OD2.7mm
- J7: value MIC -> TX LED; footprint Connector_PinHeader_2.54mm:PinHeader_1x03_P2.54mm_Vertical -> Connector_PinHeader_2.54mm:PinHeader_1x02_P2.54mm_Vertical; symbol Connector_Generic:Conn_01x03 -> Connector_Generic:Conn_01x02
- L1: value 10uH -> T30-6 17T/2T; footprint Inductor_THT:L_Axial_L9.5mm_D4.0mm_P2.54mm_Vertical_Fastron_SMCC -> Serrasoid_TRX:L_T30_3pin_Vertical; symbol Device:L -> Serrasoid_TRX:L_Tap
- L3: value T30-6 17T/2T -> 10uH; footprint Serrasoid_TRX:L_T30_3pin_Vertical -> Inductor_THT:L_Axial_L9.5mm_D4.0mm_P2.54mm_Vertical_Fastron_SMCC; symbol Serrasoid_TRX:L_Tap -> Device:L
- Q1: value 2SC1815 -> 2N3866; footprint Package_TO_SOT_THT:TO-92_Inline -> Package_TO_SOT_THT:TO-39-3; symbol Transistor_BJT:Q_NPN_ECB -> Transistor_BJT:Q_NPN_EBC
- Q2: value 2SA1015 -> RD06HHF1; footprint Package_TO_SOT_THT:TO-92_Inline -> Package_TO_SOT_THT:TO-220-3_Vertical; symbol Transistor_BJT:Q_PNP_ECB -> Serrasoid_TRX:RD_MOSFET_GSD
- Q3: value 2N7000 -> RD16HHF1; footprint Package_TO_SOT_THT:TO-92_Inline -> Package_TO_SOT_THT:TO-220-3_Vertical; symbol Transistor_FET:2N7000 -> Serrasoid_TRX:RD_MOSFET_GSD
- Q4: value 2N3866 -> 2SC1815; footprint Package_TO_SOT_THT:TO-39-3 -> Package_TO_SOT_THT:TO-92_Inline; symbol Transistor_BJT:Q_NPN_EBC -> Transistor_BJT:Q_NPN_ECB
- Q5: value RD06HHF1 -> 2N3819; footprint Package_TO_SOT_THT:TO-220-3_Vertical -> Package_TO_SOT_THT:TO-92_Inline; symbol Serrasoid_TRX:RD_MOSFET_GSD -> Transistor_FET:2N3819
- Q6: value RD16HHF1 -> 2N7000; footprint Package_TO_SOT_THT:TO-220-3_Vertical -> Package_TO_SOT_THT:TO-92_Inline; symbol Serrasoid_TRX:RD_MOSFET_GSD -> Transistor_FET:2N7000
- Q7: value 2N3819 -> 2SA1015; symbol Transistor_FET:2N3819 -> Transistor_BJT:Q_PNP_ECB
- R1: value 4.7k -> 3.9k
- R10: value 1.5k -> 1k
- R11: value 100 -> 3.3k
- R12: value 1.5k -> 100; footprint Resistor_THT:R_Axial_DIN0207_L6.3mm_D2.5mm_P2.54mm_Vertical -> Resistor_THT:R_Axial_DIN0414_L11.9mm_D4.5mm_P5.08mm_Vertical
- R13: value 10k -> 100; footprint Resistor_THT:R_Axial_DIN0207_L6.3mm_D2.5mm_P2.54mm_Vertical -> Resistor_THT:R_Axial_DIN0414_L11.9mm_D4.5mm_P5.08mm_Vertical
- R14: value 100 -> 1k
- R15: value 4.7k -> 10
- R16: value 3.9k -> 510
- R17: value 1.8k -> 3.3k
- R18: value 910 -> 1k
- R19: value 510 -> 10k
- R2: value 4.7k -> 1.8k
- R21: value 100 -> 4.7k
- R22, R64: value 10k -> 4.7k
- R24: value 470 -> 10k
- R25: value 2.2k -> 47k
- R27: value 220k -> 10k
- R28: value 100k -> 10k
- R29, R48: value 10k -> 100
- R3: value 10k -> 120
- R30: value 2.2k -> 1k
- R31: value 15k -> 10k
- R32: value 15k -> 470
- R33: value 100k -> 2.2k
- R34: value 10k -> 1.5k
- R35: value 560 -> 10k
- R36: value 120 -> 10k
- R37: value 4.7 -> 10k
- R38, R61: value 10 -> 4.7k
- R39: value 10 -> 220k
- R4: value 10k -> 560
- R40: value 47 -> 330
- R41: value 3.3k -> 1.2k
- R43: value 10 -> 100
- R44: value 100 -> 10k; footprint Resistor_THT:R_Axial_DIN0414_L11.9mm_D4.5mm_P5.08mm_Vertical -> Resistor_THT:R_Axial_DIN0207_L6.3mm_D2.5mm_P2.54mm_Vertical
- R45: footprint Resistor_THT:R_Axial_DIN0414_L11.9mm_D4.5mm_P5.08mm_Vertical -> Resistor_THT:R_Axial_DIN0207_L6.3mm_D2.5mm_P2.54mm_Vertical
- R46: value 3.3k -> 100k
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Connections:
- net +13V8: now also C26.1, C33.1, C35.1, C37.1, C4.1, C7.1, D4.1 (K), L3.1, U3.1 (IN); no longer C1.1, C2.1, C51.1, C55.1, C56.1, C57.1, D3.1 (K), L1.1, U2.1 (IN)
- net +3V3S: now also C28.1, C30.1, U7.1 (VDDO), U7.8 (VDD); no longer C12.1, C13.1, U4.1 (VO), U6.8 (VDD)
- net +3V3X: now also R19.1, R21.1, R22.1, R23.1, R26.1, R28.1, U9.10 (3V3); no longer R1.1, R2.1, R3.1, R4.1, R5.1, R6.1, U5.10 (3V3)
- net +5V: now also C18.1, C20.1, D3.2 (A), U6.3 (VI); no longer C4.1, C5.1, D2.2 (A), U1.3 (OUT)
- net +5VA: now also C55.1, C67.1, C68.2, C69.2, C71.2, C75.1, C88.1, R52.2, R56.1, U10.1 (VO), U13.8 (VCC), U14.4 (VCC)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; no longer C74.1, C77.2, C78.2, C79.2, C80.1, C89.1, C92.1, R56.2, R62.1, U14.8 (VCC), U15.4 (VCC), U17.1 (VO)
- net +5VT: now also C21.1, C25.1, C36.1, C66.1, C76.1, C8.1, C82.1, C90.1, C94.1, D9.2 (A), R32.1, R35.1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; no longer C10.1, C11.1, C17.1, C18.1, C20.1, C28.1, C29.1, C30.1, C41.1, D4.2 (A), R12.1, R15.1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
- net +8V: now also C12.1, C13.1, C14.1, U3.3 (OUT), U5.1 (IN); no longer C7.1, C8.1, C9.1, U2.3 (OUT), U3.1 (IN)
- net GND: now also C18.2, C21.2, C31.2, C35.2, C36.2, C37.2, C38.2, C39.2, C43.2, C45.2, C52.2, C58.2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; no longer C10.2, C17.2, C27.2, C3.2, C44.2, C54.2, C56.2, C59.2, C60.2, C64.2, C69.2, C70.2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
- net RX8V: now also C49.1, C50.1, C62.1, C87.1, R42.1, U10.3 (VI), U18.6 (V+); no longer C16.1, C71.1, C84.1, C88.1, R53.1, U16.6 (V+), U17.3 (VI)
- net TX8V: now also C16.1, C51.1, R11.1, R17.1, R34.1, R4.1; no longer C15.1, C47.1, R10.1, R35.1, R41.1, R46.1
- net at TP4.1: now also R1.1, U17.13 (Q), U2.1; no longer R21.1
- net at C38.1: now also L7.1, T1.3 (SA); no longer R32.2
- net at C39.1: now also R18.2, R23.2, U9.1 (D0/A0); no longer C37.2
- net at R30.2, R31.1: now also Q4.3 (B); no longer D6.2 (A), D7.1 (K)
- net at D12.1 (K), R66.1, R67.1: now also C92.1; no longer C94.1
- net at R67.2, R68.1: now also U9.3 (D2/A2); no longer U5.3 (D2/A2)
- net at C78.1: now also R55.1, U14.9 (AUDIO); no longer U15.6 (DEC1)
- net at VR3.1: now also C60.2; no longer C36.2
- net at VR3.2: now also U11.5 (+)
- net at VR2.1: now also R17.2; no longer R15.2
- net at D8.1 (K), R49.1: now also D7.2 (A), R47.2; no longer C65.1, R50.1
- net at U9.14 (D7/RX): now also R59.1; no longer C21.1
- net at L7.2, L8.1: now also C41.1; no longer C60.1
- net at L8.2, L9.1: now also C42.1; no longer C61.1
- net at L10.1, TC3.1: now also C53.1, C56.1; no longer C67.1, C68.1
- net at R29.1: now also TP1.1, U8.6; no longer R28.1
- net at R30.1: now also U9.11 (D10/MOSI); no longer R28.2
- net at R10.2: now also C17.2, R7.1, R9.1; no longer J6.1 (Pin_1)
- net at FL2.1 (IN): now also U14.3 (MIX_OUT); no longer U15.3 (MIX_OUT)
- net at FL2.3 (OUT): now also U14.5 (LIM_IN); no longer U15.5 (LIM_IN)
- net at D11.1 (K), D12.2 (A): now also C86.2; no longer C93.2
- net at K1.4: now also J6.1 (Pin_1); no longer J5.1 (Pin_1)
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Other:
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
Commit message: 受信の第 1 混合を SA612AN（製造中止）から NJM2594V に変更し、10.7MHz 増幅を追加（回路図・基板 Ver 1.1）
- U13 NJM2594V（秋月 111195、SSOP8 0.65mm）: データシートの応用回路（エミッタフォロワ出力）どおり。
  5 番 信号、6 番 バイパス、7 番 局発（R41 1.2k / R45 100Ω で約 106mVrms）、3 番 出力（R48 1k）、2・8 番 開放
  この機械で唯一の表面実装部品（ユーザーが了承）。gen_pcb.py は NJM2594V 以外の表面実装で止まる
- 変換利得 0dB（SA612 は約 +14dB）を 10.7MHz 増幅（Q6 2SC1815、約 20dB）で補う。計算は docs/回路図論理チェック.md の追補
- 部品番号を回路図の位置順に振り直し（tools/renumber.py を 2 回目に対応。対応表は今日の振り直し前との対応）
- 基板: +5VA を 0.3mm に、U13 の GND はビアで内層へ（tools/pcb_smd_gnd.py）、ケースの放熱器がかかる上辺 1.6mm を部品禁止、
  ミキサー〜増幅〜水晶フィルタをまとめて配置。残った未接続を引く tools/fix_route.py を route.sh に組み込み
- 確認: 照合 678 ピン一致、ERC 0、DRC エラー 0・未接続 0・回路図との食い違い 0（シルクの警告のみ）、ケースの干渉チェック通過
- 部品表・購入用部品表（NJM2594V は秋月）・回路図 PDF・部品実装図・A3 配置図・docx・ケースの部品位置と画像を更新

Co-Authored-By: Claude Opus 5.5 <noreply@anthropic.com>
Parts:
- added C95: 10u, Capacitor_THT:CP_Radial_D5.0mm_P2.00mm, symbol Device:C_Polarized
- added C96: 0.047u, Capacitor_THT:C_Disc_D5.0mm_W2.5mm_P2.50mm, symbol Device:C
- added C97: 0.47u, Capacitor_THT:C_Disc_D5.0mm_W2.5mm_P2.50mm, symbol Device:C
- added C98: 220u, Capacitor_THT:CP_Radial_D6.3mm_P2.50mm, symbol Device:C_Polarized
- added Q9: 2SC1815, Package_TO_SOT_THT:TO-92_Inline, symbol Transistor_BJT:Q_NPN_ECB
- added R69, R73: 10k, Resistor_THT:R_Axial_DIN0207_L6.3mm_D2.5mm_P2.54mm_Vertical, symbol Device:R
- added R70: 470k, Resistor_THT:R_Axial_DIN0207_L6.3mm_D2.5mm_P2.54mm_Vertical, symbol Device:R
- added R71: 10, Resistor_THT:R_Axial_DIN0207_L6.3mm_D2.5mm_P2.54mm_Vertical, symbol Device:R
- added R72: 100k, Resistor_THT:R_Axial_DIN0207_L6.3mm_D2.5mm_P2.54mm_Vertical, symbol Device:R
- added R74: 22k, Resistor_THT:R_Axial_DIN0207_L6.3mm_D2.5mm_P2.54mm_Vertical, symbol Device:R
- C65: value 0.01u -> 0.1u
- C68: value 0.1u -> 0.01u
- C70: value 68p -> 0.1u; footprint Capacitor_THT:C_Disc_D3.0mm_W1.6mm_P2.50mm -> Capacitor_THT:C_Disc_D5.0mm_W2.5mm_P2.50mm
- C71: value 220p -> 2.2n; footprint Capacitor_THT:C_Disc_D3.0mm_W1.6mm_P2.50mm -> Capacitor_THT:C_Disc_D5.0mm_W2.5mm_P2.50mm
- C72: value 2.2n -> 0.01u
- C77, C81: value 1u -> 0.1u
- C78: value 2.2n -> 1u
- C79: value 10u -> 68p; footprint Capacitor_THT:CP_Radial_D5.0mm_P2.00mm -> Capacitor_THT:C_Disc_D3.0mm_W1.6mm_P2.50mm; symbol Device:C_Polarized -> Device:C
- C80: value 0.047u -> 220p; footprint Capacitor_THT:C_Disc_D5.0mm_W2.5mm_P2.50mm -> Capacitor_THT:C_Disc_D3.0mm_W1.6mm_P2.50mm
- C82, C86: value 0.1u -> 10u; footprint Capacitor_THT:C_Disc_D5.0mm_W2.5mm_P2.50mm -> Capacitor_THT:CP_Radial_D5.0mm_P2.00mm; symbol Device:C -> Device:C_Polarized
- C83, C89: value 10u -> 0.1u; footprint Capacitor_THT:CP_Radial_D5.0mm_P2.00mm -> Capacitor_THT:C_Disc_D5.0mm_W2.5mm_P2.50mm; symbol Device:C_Polarized -> Device:C
- C85: value 0.1u -> 2.2n
- C87: value 100u -> 0.047u; footprint Capacitor_THT:CP_Radial_D6.3mm_P2.50mm -> Capacitor_THT:C_Disc_D5.0mm_W2.5mm_P2.50mm; symbol Device:C_Polarized -> Device:C
- C88: value 0.1u -> 1u
- C91: value 0.047u -> 0.1u
- C92: value 0.47u -> 100u; footprint Capacitor_THT:C_Disc_D5.0mm_W2.5mm_P2.50mm -> Capacitor_THT:CP_Radial_D6.3mm_P2.50mm; symbol Device:C -> Device:C_Polarized
- C93: value 220u -> 0.1u; footprint Capacitor_THT:CP_Radial_D6.3mm_P2.50mm -> Capacitor_THT:C_Disc_D5.0mm_W2.5mm_P2.50mm; symbol Device:C_Polarized -> Device:C
- Q6: value 2N7000 -> 2SC1815; symbol Transistor_FET:2N7000 -> Transistor_BJT:Q_NPN_ECB
- Q7: value 2SA1015 -> 2N7000; symbol Transistor_BJT:Q_PNP_ECB -> Transistor_FET:2N7000
- Q8: value 2SC1815 -> 2SA1015; symbol Transistor_BJT:Q_NPN_ECB -> Transistor_BJT:Q_PNP_ECB
- R48: value 100 -> 1k
- R49: value 15k -> 100
- R51: value 1.5k -> 22k
- R52: value 20k -> 4.7k
- R53, R57: value 10k -> 1.5k
- R54: value 10k -> 82
- R55: value 10k -> 180
- R56: value 10k -> 15k
- R58, R66: value 100k -> 10k
- R59: value 10k -> 20k
- R61: value 4.7k -> 100k
- R63: value 470k -> 10k
- R64: value 4.7k -> 10k
- R65: value 10 -> 4.7k
- R68: value 22k -> 4.7k
- U13: value SA612AN -> NJM2594V; footprint Package_DIP:DIP-8_W7.62mm_Socket -> Package_SO:TSSOP-8_4.4x3mm_P0.65mm; symbol Serrasoid_TRX:SA612 -> Serrasoid_TRX:NJM2594
- U14: value MC3361 -> MAX913CPA; footprint Package_DIP:DIP-16_W7.62mm_Socket -> Package_DIP:DIP-8_W7.62mm_Socket; symbol Serrasoid_TRX:MC3361 -> Comparator:LT1016
- U15: value MAX913CPA -> MC3361; footprint Package_DIP:DIP-8_W7.62mm_Socket -> Package_DIP:DIP-16_W7.62mm_Socket; symbol Comparator:LT1016 -> Serrasoid_TRX:MC3361
- U16: value MCP6002 -> 74HCT123; footprint Package_DIP:DIP-8_W7.62mm_Socket -> Package_DIP:DIP-16_W7.62mm_Socket; symbol Amplifier_Operational:MCP6002-xP -> 74xx:74HC123
- U17: value 74HCT123 -> MCP6002; footprint Package_DIP:DIP-16_W7.62mm_Socket -> Package_DIP:DIP-8_W7.62mm_Socket; symbol 74xx:74HC123 -> Amplifier_Operational:MCP6002-xP
Connections:
- net +5VA: now also C66.1, C76.2, C77.2, C80.2, C83.1, C94.1, R59.2, R64.1, U13.1 (V+), U15.4 (VCC), U17.8 (V+); no longer C67.1, C68.2, C69.2, C71.2, C75.1, C88.1, R52.2, R56.1, U13.8 (VCC), U14.4 (VCC), U16.8 (V+)
- net +5VT: now also C65.1, C75.1, C81.1, C89.1, C93.1, R57.1, R65.1, U14.1 (V+), U16.16 (VCC), U16.3 (Clr), U16.9 (A); no longer C66.1, C76.1, C82.1, C90.1, C94.1, R51.1, R64.1, U15.1 (V+), U17.16 (VCC), U17.3 (Clr), U17.9 (A)
- net GND: now also C69.2, C70.2, C81.2, C86.2, C93.2, Q7.1 (S), R48.2, R52.2, R55.2, R58.2, R60.2, U13.4 (GND), U14.4 (V-), U14.5 (LATCH), U14.6 (GND), U15.15 (GND), U16.1 (A), U16.10 (B), U16.11 (Clr), U16.8 (GND), U17.4 (V-), C95.2, C96.2, C97.2, Q9.1 (E), R69.2, R72.2, R74.2; no longer C75.2, C79.2, C80.2, C85.2, C88.2, C91.2, Q6.1 (S), Q8.1 (E), R53.2, R54.2, R62.2, R66.2, R68.2, U13.3 (GND), U14.15 (GND), U15.4 (V-), U15.5 (LATCH), U15.6 (GND), U16.4 (V-), U17.1 (A), U17.10 (B), U17.11 (Clr), U17.8 (GND)
- net RX8V: now also C69.1, C90.1, C92.1, R51.1, R53.1; no longer C85.1, C87.1
- net at R1.1, TP4.1, U2.1: now also U16.13 (Q); no longer U17.13 (Q)
- net at C78.2: now also VR5.1; no longer R57.1
- net at C57.1, D7.1 (K), D8.2 (A)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: now also C71.2; no longer C72.2
- net at D7.2 (A), D8.1 (K), R47.2: now also R50.1; no longer R49.1
- net at FL2.1 (IN): now also U15.3 (MIX_OUT); no longer U14.3 (MIX_OUT)
- net at FL2.3 (OUT): now also U15.5 (LIM_IN); no longer U14.5 (LIM_IN)
- net at D11.1 (K), D12.2 (A): now also C91.2; no longer C86.2
- net at U13.2 (OUT1): no longer C65.1
- net at C63.2: now also U13.5 (SIG); no longer U13.1 (IN_A)
- net at FL1.1 (IN): now also C72.2; no longer U13.4 (OUT_A)
- net at U13.6 (BYP): now also C67.1; no longer C64.2
- net at U13.7 (CARR): now also C64.2
- net at C91.1: now also U17.1, R70.2; no longer R65.2
- net at J8.1 (Pin_1): now also C88.2; no longer C81.2
- net at C68.1: now also R48.1, U13.3 (OUT2); no longer U14.6 (DEC1)
- net at Q6.2 (C): now also C72.1, R53.2; no longer R48.2
- net at R58.1: now also C75.2, D10.1 (K), Q8.3 (B); no longer VR5.2
- net at U14.7 (Q): now also U16.2 (B); no longer C69.1
- net at TP3.1, U11.13 (-), U11.14: now also U14.3 (-); no longer U15.3 (-)
- net at FL1.3 (OUT): now also U15.16 (MIX_IN); no longer U14.16 (MIX_IN)
- net at U12.3 (Q0): now also R49.1; no longer R48.1
- net at VR4.2, VR4.3: now also Q8.1 (E); no longer Q7.1 (E)
- net at U17.5 (+): now also C86.1, R60.1, R64.2, U17.3 (+)
- net at U17.6 (-): now also U17.7
- net at R61.1: now also VR5.2; no longer J8.2 (Pin_2)
- net at C74.2, U11.8, U11.9 (-): now also C78.1; no longer C77.1
- net at R51.2: now also C68.2, Q6.3 (B), R52.1; no longer VR4.1
- net at U16.6 (Cext): no longer U16.7
- net at VR7.1: now also R65.2; no longer R64.2
- net at C84.2, VR7.2, VR7.3: now also U16.15 (RCext); no longer U17.15 (RCext)
- net at C84.1: now also U16.14 (Cext); no longer U17.14 (Cext)
- net at U17.2 (-): now also R66.2, R70.1; no longer U15.7 (Q)
- net at J9.1 (Pin_1): now also C98.2; no longer C93.2
- net at U15.8 (QUAD): now also R59.1, X2.1
- net at U9.14 (D7/RX): now also R67.1; no longer R59.1
- net at U18.7 (BYPASS): now also C95.1; no longer C89.1
- new net: Q9.3 (B), R67.2, R69.1
- new net: C98.1, R71.1, U18.5
- new net: C74.1, R50.2, R56.1
- new net: C71.1, R56.2, U11.10 (+)
- new net: C85.1, R63.1, U15.9 (AUDIO)
- new net: C85.2, R66.1
- new net: C96.1, R71.2
- new net: C97.1, D12.1 (K), R72.1, R73.1
- new net: R73.2, R74.1, U9.3 (D2/A2)
- new net: Q6.1 (E), R54.1
- new net: Q7.2 (G), R49.2
- new net: C87.1, C88.1, R63.2
- new net: C76.1, U15.6 (DEC1)
- new net: C73.1, Q7.3 (D), Q8.2 (C), TP2.1, U14.2 (+)
- new net: R61.2, R62.2, U11.12 (+)
- new net: J8.2 (Pin_2), R68.1
- new net: Q9.2 (C), R68.2, U18.3 (+)
- new net: R57.2, VR4.1
- new net: C79.1, U15.1 (OSC_B), X1.1
- new net: C82.1, R62.1, VR6.2
- new net: C79.2, C80.1, U15.2 (OSC_E)
- new net: C70.1, R54.2, R55.1
- new net: C77.1, U15.7 (DEC2)
- now unconnected: U14.8 (QUAD), U16.5 (+)
Other:
- note added: "送信: マイク → 送信音声 → セラゾイド変調（915.625kHz で PM）→ 逓倍 ×32 → 送信RF（10W）→ ANT 受信: ANT → 受信（2N3819 → NJM2594 → 10.7MHz 増幅 → 10.7MHz → MC3361 → LM386）→ SP 制御: XIAO ESP32C3 ＋ Si5351（CLK0 = 変調基準 9.15625MHz、CLK1 = 受信局発 18.6MHz） ブロックの中もブロックの間も線で結線（電源も線。電源の名前は出どころの電源記号で示す。GND だけ GND 記号）"
- note removed: "送信: マイク → 送信音声 → セラゾイド変調（915.625kHz で PM）→ 逓倍 ×32 → 送信RF（10W）→ ANT 受信: ANT → 受信（2N3819 → SA612 → 10.7MHz → MC3361 → LM386）→ SP 制御: XIAO ESP32C3 ＋ Si5351（CLK0 = 変調基準 9.15625MHz、CLK1 = 受信局発 18.6MHz） ブロックの中もブロックの間も線で結線（電源も線。電源の名前は出どころの電源記号で示す。GND だけ GND 記号）"
- moved on the sheet: C65, C66, C67, C68, C69, C70, C71, C72, C75, C76, C77, C78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

Commit message: スプリアス対策: 逓倍を ×16 にし、段間同調と PLL 追従フィルタを追加（回路図・基板 Ver 1.2）
Ver 1.1（915.625kHz × 32、段間に同調なし）は計算でアンテナ端 −13.5dBc（27.47MHz）の側帯波が出て、
規格（30MHz 以下: 50mW 以下かつ −50dBc）を満たさなかった。次の 3 つを入れ、計算では最悪 −99dBc。

- 逓倍数を減らす: CLK0 18.3125MHz ÷10 = 1.83125MHz、×16（4 段）。C71 68p、ワンショット 2.2k＋VR 5k（273ns）
- 段間同調: 段 1〜3 の後に LC 並列共振（10µH/180p・4.7µH/100p・1µH/120p、Q 約 5、調整なし）
  → 74HCU04 自己バイアス → 74AC14
- PLL（新ブロック）: 74AC74・74AC00 の位相周波数比較、MCP6002 の差動積分、VCO 専用 74HCU04 の LC 発振
  （T50-6 15T、1N4007 を可変容量に）。送信は 3 回路を 330Ω ずつで合成。受信中は Q3 で VCO を止める
- 送信 BPF の段間結合 2pF → 1pF（過結合で ±1.8MHz が落ちなかった）
- 基板 170×130 → 170×140mm、区画を割り直し、後面 DC ジャックの下を部品禁止。
  DRC エラー 0・未接続 0・回路図との食い違い 0、ERC 0、照合 835 ピン一致
- 部品番号を位置順に振り直し（kicad/refdes_map_2026-10-29.csv）。取り外した部品は REMOVED() で仮番号を保持
- 資料: README、回路図論理チェック・基板チェックの追補、動作説明 docx（段間同調・PLL の章）、部品実装図 9 ページ、
  A3 配置図、回路図 PDF、部品表・購入用部品表（新部品は秋月の商品ページで確認）、ケース scad・底板 STL・内部プレビュー

Co-Authored-By: Claude Opus 5.5 <noreply@anthropic.com>
Parts:
- removed unit 5 of U1
- removed unit 6 of U1
- removed unit 4 of U1
- removed unit 7 of U1
- removed unit 2 of U17
- removed unit 3 of U17
- removed unit 2 of U2
- removed unit 5 of U2
- removed unit 4 of U2
- removed unit 3 of U2
- removed unit 2 of U8
- removed unit 3 of U8
- removed unit 5 of U8
- removed unit 4 of U8
- added C100, C103, C116: 0.01u, Capacitor_THT:C_Disc_D5.0mm_W2.5mm_P2.50mm, symbol Device:C
- added C101, C102, C107, C117, C99: 0.1u, Capacitor_THT:C_Disc_D5.0mm_W2.5mm_P2.50mm, symbol Device:C
- added C104: 220u, Capacitor_THT:CP_Radial_D8.0mm_P3.50mm, symbol Device:C_Polarized
- added C105, C112, C114: 100p, Capacitor_THT:C_Disc_D3.0mm_W1.6mm_P2.50mm, symbol Device:C
- added C106: 47p, Capacitor_THT:C_Disc_D3.0mm_W1.6mm_P2.50mm, symbol Device:C
- added C108, C111: 120p, Capacitor_THT:C_Disc_D5.0mm_W2.5mm_P5.00mm, symbol Device:C
- added C109, C110: 220p, Capacitor_THT:C_Disc_D5.0mm_W2.5mm_P5.00mm, symbol Device:C
- added C113: 4.7p, Capacitor_THT:C_Disc_D3.0mm_W1.6mm_P2.50mm, symbol Device:C
- added C115: 1000p, Capacitor_THT:C_Disc_D3.0mm_W1.6mm_P2.50mm, symbol Device:C
- added D13: 1N60, Diode_THT:D_DO-35_SOD27_P2.54mm_Vertical_AnodeUp, symbol Device:D
- added L13, L15: T50-6 9T, Serrasoid_TRX:L_T50_2pin_Vertical, symbol Device:L
- added L14: T50-6 10T, Serrasoid_TRX:L_T50_2pin_Vertical, symbol Device:L
- added L16: 4.7uH, Inductor_THT:L_Axial_L9.5mm_D4.0mm_P2.54mm_Vertical_Fastron_SMCC, symbol Device:L
- added Q10: RD16HHF1, Package_TO_SOT_THT:TO-220-3_Vertical, symbol Serrasoid_TRX:RD_MOSFET_GSD
- added R75, R83: 10, Resistor_THT:R_Axial_DIN0207_L6.3mm_D2.5mm_P2.54mm_Vertical, symbol Device:R
- added R76, R78, R82, R89: 1k, Resistor_THT:R_Axial_DIN0207_L6.3mm_D2.5mm_P2.54mm_Vertical, symbol Device:R
- added R77, R86: 3.3k, Resistor_THT:R_Axial_DIN0207_L6.3mm_D2.5mm_P2.54mm_Vertical, symbol Device:R
- added R79: 470, Resistor_THT:R_Axial_DIN0207_L6.3mm_D2.5mm_P2.54mm_Vertical, symbol Device:R
- added R80, R81: 100, Resistor_THT:R_Axial_DIN0414_L11.9mm_D4.5mm_P5.08mm_Vertical, symbol Device:R
- added R84, R85, R91: 1M, Resistor_THT:R_Axial_DIN0207_L6.3mm_D2.5mm_P2.54mm_Vertical, symbol Device:R
- added R87: 910, Resistor_THT:R_Axial_DIN0207_L6.3mm_D2.5mm_P2.54mm_Vertical, symbol Device:R
- added R88: 330, Resistor_THT:R_Axial_DIN0207_L6.3mm_D2.5mm_P2.54mm_Vertical, symbol Device:R
- added R90, R93: 10k, Resistor_THT:R_Axial_DIN0207_L6.3mm_D2.5mm_P2.54mm_Vertical, symbol Device:R
- added R92: 47k, Resistor_THT:R_Axial_DIN0207_L6.3mm_D2.5mm_P2.54mm_Vertical, symbol Device:R
- added TC5: 30p, Serrasoid_TRX:C_Trimmer_TMCV01, symbol Device:C_Trim
- added TP5: PM, TestPoint:TestPoint_THTPad_D1.5mm_Drill0.7mm, symbol Connector:TestPoint
- added TP6: X16, TestPoint:TestPoint_THTPad_D1.5mm_Drill0.7mm, symbol Connector:TestPoint
- added unit 6 of U11
- added unit 7 of U11
- added unit 2 of U14
- added unit 3 of U14
- added unit 5 of U16
- added unit 4 of U16
- added U19: 74HCT123, Package_DIP:DIP-16_W7.62mm_Socket, symbol 74xx:74HC123
- added U20, U23: 74AC14, Package_DIP:DIP-14_W7.62mm_Socket, symbol 74xx:74HC14
- added U21: 74AC86, Package_DIP:DIP-14_W7.62mm_Socket, symbol 74xx:74HC86
- added U22: 74HCU04, Package_DIP:DIP-14_W7.62mm_Socket, symbol 74xx:74HC04
- added unit 2 of U3
- added unit 5 of U3
- added unit 4 of U3
- added unit 3 of U3
- added unit 3 of U7
- added unit 2 of U7
- C1, C73, C9: value 100p -> 0.1u; footprint Capacitor_THT:C_Disc_D3.0mm_W1.6mm_P2.50mm -> Capacitor_THT:C_Disc_D5.0mm_W2.5mm_P2.50mm
- C10: value 0.01u -> 22p; footprint Capacitor_THT:C_Disc_D5.0mm_W2.5mm_P2.50mm -> Capacitor_THT:C_Disc_D3.0mm_W1.6mm_P2.50mm
- C12: value 10u -> 220p; footprint Capacitor_THT:CP_Radial_D5.0mm_P2.00mm -> Capacitor_THT:C_Disc_D3.0mm_W1.6mm_P2.50mm; symbol Device:C_Polarized -> Device:C
- C13, C66: value 0.1u -> 220p; footprint Capacitor_THT:C_Disc_D5.0mm_W2.5mm_P2.50mm -> Capacitor_THT:C_Disc_D3.0mm_W1.6mm_P2.50mm
- C14, C22, C65, C7: value 0.1u -> 10u; footprint Capacitor_THT:C_Disc_D5.0mm_W2.5mm_P2.50mm -> Capacitor_THT:CP_Radial_D5.0mm_P2.00mm; symbol Device:C -> Device:C_Polarized
- C15, C16, C17, C27, C32, C68: value 0.01u -> 0.1u
- C18, C21, C82, C86: value 10u -> 0.01u; footprint Capacitor_THT:CP_Radial_D5.0mm_P2.00mm -> Capacitor_THT:C_Disc_D5.0mm_W2.5mm_P2.50mm; symbol Device:C_Polarized -> Device:C
- C19: value 0.01u -> 10u; footprint Capacitor_THT:C_Disc_D5.0mm_W2.5mm_P2.50mm -> Capacitor_THT:CP_Radial_D5.0mm_P2.00mm; symbol Device:C -> Device:C_Polarized
- C2: value 22p -> 470u; footprint Capacitor_THT:C_Disc_D3.0mm_W1.6mm_P2.50mm -> Capacitor_THT:CP_Radial_D8.0mm_P3.50mm; symbol Device:C -> Device:C_Polarized
- C23, C45: value 100p -> 0.01u; footprint Capacitor_THT:C_Disc_D3.0mm_W1.6mm_P2.50mm -> Capacitor_THT:C_Disc_D5.0mm_W2.5mm_P2.50mm
- C25, C26, C34, C90: value 0.1u -> 0.01u
- C29: value 0.01u -> 470p; footprint Capacitor_THT:C_Disc_D5.0mm_W2.5mm_P2.50mm -> Capacitor_THT:C_Disc_D3.0mm_W1.6mm_P2.50mm
- C3, C56: value 2p -> 0.1u; footprint Capacitor_THT:C_Disc_D3.0mm_W1.6mm_P2.50mm -> Capacitor_THT:C_Disc_D5.0mm_W2.5mm_P2.50mm
- C31: value 82p -> 0.1u; footprint Capacitor_THT:C_Disc_D3.0mm_W1.6mm_P2.50mm -> Capacitor_THT:C_Disc_D5.0mm_W2.5mm_P2.50mm
- C35: value 0.01u -> 47p; footprint Capacitor_THT:C_Disc_D5.0mm_W2.5mm_P2.50mm -> Capacitor_THT:C_Disc_D3.0mm_W1.6mm_P2.50mm
- C37: value 220u -> 0.1u; footprint Capacitor_THT:CP_Radial_D8.0mm_P3.50mm -> Capacitor_THT:C_Disc_D5.0mm_W2.5mm_P2.50mm; symbol Device:C_Polarized -> Device:C
- C38: value 120p -> 0.01u; footprint Capacitor_THT:C_Disc_D5.0mm_W2.5mm_P5.00mm -> Capacitor_THT:C_Disc_D5.0mm_W2.5mm_P2.50mm
- C39: value 0.01u -> 27p; footprint Capacitor_THT:C_Disc_D5.0mm_W2.5mm_P2.50mm -> Capacitor_THT:C_Disc_D3.0mm_W1.6mm_P2.50mm
- C4: value 470u -> 22p; footprint Capacitor_THT:CP_Radial_D8.0mm_P3.50mm -> Capacitor_THT:C_Disc_D3.0mm_W1.6mm_P2.50mm; symbol Device:C_Polarized -> Device:C
- C40: value 47p -> 0.1u; footprint Capacitor_THT:C_Disc_D3.0mm_W1.6mm_P2.50mm -> Capacitor_THT:C_Disc_D5.0mm_W2.5mm_P2.50mm
- C41: value 220p -> 0.1u; footprint Capacitor_THT:C_Disc_D5.0mm_W2.5mm_P5.00mm -> Capacitor_THT:C_Disc_D5.0mm_W2.5mm_P2.50mm
- C42: value 220p -> 68p; footprint Capacitor_THT:C_Disc_D5.0mm_W2.5mm_P5.00mm -> Capacitor_THT:C_Disc_D3.0mm_W1.6mm_P2.50mm
- C43: value 120p -> 220p; footprint Capacitor_THT:C_Disc_D5.0mm_W2.5mm_P5.00mm -> Capacitor_THT:C_Disc_D3.0mm_W1.6mm_P2.50mm
- C44: value 4.7p -> 0.01u; footprint Capacitor_THT:C_Disc_D3.0mm_W1.6mm_P2.50mm -> Capacitor_THT:C_Disc_D5.0mm_W2.5mm_P2.50mm
- C46: value 0.01u -> 56p; footprint Capacitor_THT:C_Disc_D5.0mm_W2.5mm_P2.50mm -> Capacitor_THT:C_Disc_D3.0mm_W1.6mm_P2.50mm
- C48: value 0.01u -> 2.2n
- C49: value 47u -> 10u
- C5: value 22p -> 0.33u; footprint Capacitor_THT:C_Disc_D3.0mm_W1.6mm_P2.50mm -> Capacitor_THT:C_Disc_D5.0mm_W2.5mm_P2.50mm
- C50: value 0.1u -> 0.047u
- C51: value 47u -> 1u; footprint Capacitor_THT:CP_Radial_D5.0mm_P2.00mm -> Capacitor_THT:C_Disc_D5.0mm_W2.5mm_P2.50mm; symbol Device:C_Polarized -> Device:C
- C52: value 47u -> 0.1u; footprint Capacitor_THT:CP_Radial_D5.0mm_P2.00mm -> Capacitor_THT:C_Disc_D5.0mm_W2.5mm_P2.50mm; symbol Device:C_Polarized -> Device:C
- C53: value 22p -> 0.01u; footprint Capacitor_THT:C_Disc_D3.0mm_W1.6mm_P2.50mm -> Capacitor_THT:C_Disc_D5.0mm_W2.5mm_P2.50mm
- C54, C78: value 1u -> 0.1u
- C55: value 10u -> 100u; footprint Capacitor_THT:CP_Radial_D5.0mm_P2.00mm -> Capacitor_THT:CP_Radial_D6.3mm_P2.50mm
- C58: value 22p -> 0.047u; footprint Capacitor_THT:C_Disc_D3.0mm_W1.6mm_P2.50mm -> Capacitor_THT:C_Disc_D5.0mm_W2.5mm_P2.50mm
- C59: value 220p -> 0.47u; footprint Capacitor_THT:C_Disc_D3.0mm_W1.6mm_P2.50mm -> Capacitor_THT:C_Disc_D5.0mm_W2.5mm_P2.50mm
- C6: value 0.33u -> 0.1u
- C60: value 1u -> 220u; footprint Capacitor_THT:C_Disc_D5.0mm_W2.5mm_P2.50mm -> Capacitor_THT:CP_Radial_D6.3mm_P2.50mm; symbol Device:C -> Device:C_Polarized
- C61, C63, C64: value 0.01u -> 47u; footprint Capacitor_THT:C_Disc_D5.0mm_W2.5mm_P2.50mm -> Capacitor_THT:CP_Radial_D5.0mm_P2.00mm; symbol Device:C -> Device:C_Polarized
- C62, C72: value 0.01u -> 1u
- C67: value 0.1u -> 1u
- C69: value 0.1u -> 2.2n
- C70: value 0.1u -> 4.7n
- C71: value 2.2n -> 68p; footprint Capacitor_THT:C_Disc_D5.0mm_W2.5mm_P2.50mm -> Capacitor_THT:C_Disc_D3.0mm_W1.6mm_P2.50mm
- C74: value 4.7n -> 10u; footprint Capacitor_THT:C_Disc_D5.0mm_W2.5mm_P2.50mm -> Capacitor_THT:CP_Radial_D5.0mm_P2.00mm; symbol Device:C -> Device:C_Polarized
- C76, C83: value 0.1u -> 100p; footprint Capacitor_THT:C_Disc_D5.0mm_W2.5mm_P2.50mm -> Capacitor_THT:C_Disc_D3.0mm_W1.6mm_P2.50mm
- C79: value 68p -> 22p
- C8: value 0.1u -> 2p; footprint Capacitor_THT:C_Disc_D5.0mm_W2.5mm_P2.50mm -> Capacitor_THT:C_Disc_D3.0mm_W1.6mm_P2.50mm
- C80: value 220p -> 1p
- C81: value 0.1u -> 22p; footprint Capacitor_THT:C_Disc_D5.0mm_W2.5mm_P2.50mm -> Capacitor_THT:C_Disc_D3.0mm_W1.6mm_P2.50mm
- C84: value 100p -> 82p
- C85: value 2.2n -> 0.01u
- C87, C96: value 0.047u -> 0.01u
- C88: value 1u -> 0.01u
- C92: value 100u -> 0.01u; footprint Capacitor_THT:CP_Radial_D6.3mm_P2.50mm -> Capacitor_THT:C_Disc_D5.0mm_W2.5mm_P2.50mm; symbol Device:C_Polarized -> Device:C
- C94: value 0.1u -> 180p; footprint Capacitor_THT:C_Disc_D5.0mm_W2.5mm_P2.50mm -> Capacitor_THT:C_Disc_D3.0mm_W1.6mm_P2.50mm
- C95: value 10u -> 120p; footprint Capacitor_THT:CP_Radial_D5.0mm_P2.00mm -> Capacitor_THT:C_Disc_D3.0mm_W1.6mm_P2.50mm; symbol Device:C_Polarized -> Device:C
- C97: value 0.47u -> 1000p; footprint Capacitor_THT:C_Disc_D5.0mm_W2.5mm_P2.50mm -> Capacitor_THT:C_Disc_D3.0mm_W1.6mm_P2.50mm
- C98: value 220u -> 1000p; footprint Capacitor_THT:CP_Radial_D6.3mm_P2.50mm -> Capacitor_THT:C_Disc_D3.0mm_W1.6mm_P2.50mm; symbol Device:C_Polarized -> Device:C
- D11, D12, D2: value 1N60 -> 1N4148; symbol Device:D -> Diode:1N4148
- D3: value 1N5819 -> 1N4148; footprint Diode_THT:D_DO-41_SOD81_P5.08mm_Vertical_AnodeUp -> Diode_THT:D_DO-35_SOD27_P2.54mm_Vertical_AnodeUp; symbol Diode:1N5819 -> Diode:1N4148
- D4: value 1N4001 -> 1N4007; symbol Diode:1N4001 -> Diode:1N4007
- D5: value 1N4148 -> 1N5819; footprint Diode_THT:D_DO-35_SOD27_P2.54mm_Vertical_AnodeUp -> Diode_THT:D_DO-41_SOD81_P5.08mm_Vertical_AnodeUp; symbol Diode:1N4148 -> Diode:1N5819
- D6, D7: value 1N4148 -> 1N60; symbol Diode:1N4148 -> Device:D
- D8: value 1N4148 -> 1N4001; footprint Diode_THT:D_DO-35_SOD27_P2.54mm_Vertical_AnodeUp -> Diode_THT:D_DO-41_SOD81_P5.08mm_Vertical_AnodeUp; symbol Diode:1N4148 -> Diode:1N4001
- J4: value ENC -> VOL; footprint Connector_PinHeader_2.54mm:PinHeader_1x05_P2.54mm_Vertical -> Connector_PinHeader_2.54mm:PinHeader_1x03_P2.54mm_Vertical; symbol Connector_Generic:Conn_01x05 -> Connector_Generic:Conn_01x03
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Connections:
- net +13V8: now also C2.1, C5.1, C91.1, D8.1 (K), L12.1, L2.1, L9.1, U4.1 (IN), C101.1, C103.1, C104.1; no longer C26.1, C33.1, C35.1, C37.1, C4.1, C7.1, D4.1 (K), L3.1, L5.1, L6.1, U3.1 (IN)
- net +3V3S: now also U10.1 (VDDO), U10.8 (VDD), U8.1 (VO); no longer U6.1 (VO), U7.1 (VDDO), U7.8 (VDD)
- net +3V3X: now also R29.1, R41.1, R42.1, U13.10 (3V3); no longer R19.1, R21.1, R22.1, U9.10 (3V3)
- net +5V: now also C19.1, D5.2 (A), U5.3 (OUT), U8.3 (VI); no longer C18.1, D3.2 (A), U4.3 (OUT), U6.3 (VI)
- net +5VA: now also C32.1, C40.2, C41.2, C43.2, C47.1, C56.1, C7.1, R25.2, R32.1, U12.4 (VCC), U2.1 (VO), U9.1 (V+)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; no longer C55.1, C66.1, C76.2, C77.2, C80.2, C83.1, C94.1, R59.2, R64.1, U10.1 (VO), U13.1 (V+), U15.4 (VCC)
- net +5VT: now also C1.1, C15.1, C27.1, C31.1, C68.1, C73.1, C77.1, C78.1, C9.1, D11.2 (A), R49.1, R51.1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; no longer C21.1, C25.1, C36.1, C65.1, C8.1, C81.1, D9.2 (A), R32.1, R35.1, R57.1, R65.1, U11.4 (V+)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
- net +8V: now also C16.1, C17.1, U4.3 (OUT), U6.1 (IN); no longer C12.1, C13.1, U3.3 (OUT), U5.1 (IN)
- net GND: now also C10.2, C17.2, C27.2, C3.2, C44.2, C56.2, C59.2, C63.2, C64.2, C68.2, C71.2, C74.2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; no longer C21.2, C25.2, C26.2, C35.2, C38.2, C40.2, C41.2, C42.2, C43.2, C45.2, C51.2, C53.2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
- net RX8V: now also C24.1, C3.1, C36.1, C52.1, C55.1, C63.1, L4.1, R15.1, R17.1, R20.1, R9.1, U15.6 (V+)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; no longer C49.1, C50.1, C62.1, C69.1, C90.1, C92.1, L12.1, R42.1, R51.1, R53.1, U10.3 (VI), U18.6 (V+)
- net TX8V: now also C64.1, C86.1, L8.1, R53.1, R71.1, R77.1, R86.1; no longer C16.1, C51.1, L4.1, R11.1, R17.1, R34.1, R4.1
- net at TP1.1: now also C29.1, R12.2, R13.1; no longer R29.1
- net at VR5.1: now also R67.2; no longer C78.2
- net at C98.2: now also R85.1, U22.5; no longer J9.1 (Pin_1)
- net at VR3.1: now also C72.2; no longer C60.2
- net at VR3.2: now also R65.1; no longer U11.5 (+)
- net at VR2.1: now also R63.2; no longer R17.2
- net at C67.1: now also C66.2, R55.2, U16.1; no longer U13.6 (BYP)
- net at C40.1: now also U12.6 (DEC1); no longer R20.2
- net at FL2.1 (IN): now also U12.3 (MIX_OUT); no longer U15.3 (MIX_OUT)
- net at FL2.3 (OUT): now also U12.5 (LIM_IN); no longer U15.5 (LIM_IN)
- net at D11.1 (K), D12.2 (A): no longer C91.2
- net at R30.1: now also R24.2, U11.11, U11.2, U11.3, U11.5, U11.9; no longer U9.11 (D10/MOSI)
- net at J6.1 (Pin_1): now also C60.2; no longer K1.4
- net at R66.1: now also C74.1, VR4.2; no longer C85.2
- net at R15.2: now also C34.2, Q2.3 (B), R16.1; no longer Q3.1 (G)
- net at R2.1: now also U1.9 (Q), U3.2; no longer U2.3
- net at R8.1: now also U10.6 (CLK1)
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Other:
- note added: "PLL"
- note added: "送信: マイク → 送信音声 → セラゾイド変調（1.83125MHz で PM）→ 逓倍 ×16（段間同調）→ PLL（VCO 29.3MHz）→ 送信RF（10W）→ ANT 受信: ANT → 受信（2N3819 → NJM2594 → 10.7MHz 増幅 → 10.7MHz → MC3361 → LM386）→ SP 制御: XIAO ESP32C3 ＋ Si5351（CLK0 = 変調基準 18.3125MHz、CLK1 = 受信局発 18.6MHz） ブロックの中もブロックの間も線で結線（電源も線。電源の名前は出どころの電源記号で示す。GND だけ GND 記号）"
- note removed: "送信: マイク → 送信音声 → セラゾイド変調（915.625kHz で PM）→ 逓倍 ×32 → 送信RF（10W）→ ANT 受信: ANT → 受信（2N3819 → NJM2594 → 10.7MHz 増幅 → 10.7MHz → MC3361 → LM386）→ SP 制御: XIAO ESP32C3 ＋ Si5351（CLK0 = 変調基準 9.15625MHz、CLK1 = 受信局発 18.6MHz） ブロックの中もブロックの間も線で結線（電源も線。電源の名前は出どころの電源記号で示す。GND だけ GND 記号）"
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
Commit message: スケッチを追加（Nextion / TJC 両対応、アナログ S メーター、周波数スキャン）
- firmware/Serrasoid_TRX/Serrasoid_TRX.ino（XIAO ESP32C3、コンパイル確認のみ・実機未確認）
  - Si5351: CLK0 = 送信周波数 × 10 ÷ 16（送信中だけ）、CLK1 = 受信周波数 − 10.7MHz（受信中だけ）
  - PTT: 局発を止める → リレー → 15ms → 変調基準。29.000〜29.700MHz の外では送信しない
  - 操作: ダイヤル = 周波数、押す = メニュー（STEP / SQL / SCAN / EXIT）、長押し = 呼出 29.300MHz
  - スキャン: 10kHz ずつ、スケルチが開いたら止まり、信号が消えて 3 秒で再開
  - S メーターは RSSI がないのでスケルチ用ノイズの減り方から換算（目安、S5 前後で頭打ち）、送信中は出力 W
- firmware/Serrasoid_TRX/nextion/: 背景画像（S メーター＋出力 W の目盛り）、表示の見本、画面データ作成手順
  （Nextion NX4832T035 = Nextion Editor、TJC4832T135 = USART HMI。スケッチは共通。.HMI / .tft は未作成）
- 表示器を Nextion NX4832T035（PSN_TRX と同じ）に、TJC4832T135 も可。J3 の値 TJC → LCD
  （2 番 = XIAO の TX → 表示器の RX（黄））。部品表・購入用部品表・README・ケースの説明を更新
- 回路図 ERC 0・照合 835 ピン一致、基板 DRC エラー 0・未接続 0・食い違い 0

Co-Authored-By: Claude Opus 5.5 <noreply@anthropic.com>
Parts:
- J3: value TJC -> LCD
