File: kicad/Serrasoid_TRX.kicad_sch (KiCad schematic)
At the start: 305 parts, among them J1 DC 13.8V, J2 I2C, J3 LCD, J4 VOL, J5 ENC, J6 SP, J7 MIC, J8 ANT, J9 TX LED, K1 G5V-2 DC12, Q1 2N3819, Q10 RD16HHF1, Q2 2SC1815, Q3 2SC1815, Q4 2SC1815, Q5 2SC1815, Q6 2N7000, Q7 2SA1015, Q8 2N3866, Q9 RD06HHF1, T1 BN43-202 2T:5T, U1 74AC74, U10 AE-Si5351A, U11 74HCU04, U12 MC3361, U13 XIAO ESP32C3, U14 MCP6002, U15 LM386N-1, U16 MCP6004, U17 74HCT4017, U18 MAX913CPA, U19 74HCT123, U2 78L05, U20 74AC14, U21 74AC86, U22 74HCU04, U23 74AC14, U3 74AC00, U4 L7808, U5 R-78E5.0-1.0, U6 L7805, U7 MCP6002, U8 LP2950-3.3, U9 NJM2594V, X1 10.245MHz, X2 CDBM455C24

Commit message: S メーターを追加（AD8307 対数増幅 ＋ ADS1115 モジュール）、基板 170 × 150mm
MC3361 に RSSI 出力がなく、ノイズの減り方からの S 表示は S5 前後で頭打ちだったため。

- 受信: IF1（10.7MHz 水晶フィルタの出力）→ R1 2.2k → Q1 2SC1815 同調増幅（L3 4.7µH・C23 47p、約 26dB）
  → U9 AD8307ANZ（DIP-8、25mV/dB、+5VA）→ RSSI_V。計算で S9 ≒ 1.27V、S2〜S9＋40 程度
- 制御: U13 ADS1115 モジュール（Adafruit 1085 と同じピン並び、I2C 0x48、A0）。XIAO の空きピンがないため I2C で読む
- 記号 AD8307・ADS1115_Module と、モジュールの外形まで取ったフットプリント ADS1115_Module_Socket を追加（mklib.py）
- 基板 170 × 140 → 150mm、区画を割り直し。DRC エラー 0・未接続 0・回路図との食い違い 0、ERC 0・照合 888 ピン一致
- ケース: pcb_v 150、背の高い部品の位置を更新（ADS1115 モジュールを追加）、assert 通過、底板 STL・内部プレビュー
- スケッチ: ADS1115 から S メーター（RSSI_MV_S9 で合わせる、S9＋20 表示）、ないときはノイズ換算に切り替え
- 部品番号を位置順に振り直し（refdes_map_2026-10-29.csv）。部品表・購入用部品表・README・回路図論理チェック／
  基板チェックの追補・部品実装図・A3 配置図・回路図 PDF・docx・LCD 画面の手順書を更新

Co-Authored-By: Claude Opus 5.5 <noreply@anthropic.com>
Parts:
- removed unit 3 of U11
- removed unit 6 of U11
- removed unit 4 of U11
- removed unit 5 of U11
- removed unit 2 of U11
- removed unit 7 of U11
- removed unit 2 of U14
- removed unit 3 of U14
- removed unit 5 of U16
- removed unit 4 of U16
- removed unit 2 of U19
- removed unit 3 of U19
- removed unit 4 of U20
- removed unit 3 of U20
- removed unit 6 of U20
- removed unit 7 of U20
- removed unit 2 of U20
- removed unit 5 of U20
- removed unit 4 of U21
- removed unit 5 of U21
- removed unit 7 of U23
- removed unit 6 of U23
- added C118, C119: 220p, Capacitor_THT:C_Disc_D5.0mm_W2.5mm_P5.00mm, symbol Device:C
- added C120: 120p, Capacitor_THT:C_Disc_D5.0mm_W2.5mm_P5.00mm, symbol Device:C
- added C121, C123: 100p, Capacitor_THT:C_Disc_D3.0mm_W1.6mm_P2.50mm, symbol Device:C
- added C122: 4.7p, Capacitor_THT:C_Disc_D3.0mm_W1.6mm_P2.50mm, symbol Device:C
- added C124: 1000p, Capacitor_THT:C_Disc_D3.0mm_W1.6mm_P2.50mm, symbol Device:C
- added C125: 0.01u, Capacitor_THT:C_Disc_D5.0mm_W2.5mm_P2.50mm, symbol Device:C
- added C126: 0.1u, Capacitor_THT:C_Disc_D5.0mm_W2.5mm_P2.50mm, symbol Device:C
- added L17: 4.7uH, Inductor_THT:L_Axial_L9.5mm_D4.0mm_P2.54mm_Vertical_Fastron_SMCC, symbol Device:L
- added Q11: RD16HHF1, Package_TO_SOT_THT:TO-220-3_Vertical, symbol Serrasoid_TRX:RD_MOSFET_GSD
- added R94: 330, Resistor_THT:R_Axial_DIN0207_L6.3mm_D2.5mm_P2.54mm_Vertical, symbol Device:R
- added R95: 1k, Resistor_THT:R_Axial_DIN0207_L6.3mm_D2.5mm_P2.54mm_Vertical, symbol Device:R
- added R96, R99: 10k, Resistor_THT:R_Axial_DIN0207_L6.3mm_D2.5mm_P2.54mm_Vertical, symbol Device:R
- added R97: 1M, Resistor_THT:R_Axial_DIN0207_L6.3mm_D2.5mm_P2.54mm_Vertical, symbol Device:R
- added R98: 47k, Resistor_THT:R_Axial_DIN0207_L6.3mm_D2.5mm_P2.54mm_Vertical, symbol Device:R
- added unit 6 of U12
- added unit 4 of U12
- added unit 7 of U12
- added unit 5 of U12
- added unit 2 of U12
- added unit 3 of U12
- added unit 4 of U18
- added unit 5 of U18
- added unit 3 of U18
- added unit 2 of U18
- added U24: 74HCU04, Package_DIP:DIP-14_W7.62mm_Socket, symbol 74xx:74HC04
- added U25: 74AC14, Package_DIP:DIP-14_W7.62mm_Socket, symbol 74xx:74HC14
- C10: value 22p -> 0.1u; footprint Capacitor_THT:C_Disc_D3.0mm_W1.6mm_P2.50mm -> Capacitor_THT:C_Disc_D5.0mm_W2.5mm_P2.50mm
- C100, C116, C18, C24, C34, C38, C45, C82, C86, C87: value 0.01u -> 0.1u
- C101, C20, C27, C30, C31, C32, C33, C47, C54, C91, C99: value 0.1u -> 0.01u
- C103: value 0.01u -> 180p; footprint Capacitor_THT:C_Disc_D5.0mm_W2.5mm_P2.50mm -> Capacitor_THT:C_Disc_D3.0mm_W1.6mm_P2.50mm
- C104: value 220u -> 120p; footprint Capacitor_THT:CP_Radial_D8.0mm_P3.50mm -> Capacitor_THT:C_Disc_D3.0mm_W1.6mm_P2.50mm; symbol Device:C_Polarized -> Device:C
- C105, C112: value 100p -> 0.01u; footprint Capacitor_THT:C_Disc_D3.0mm_W1.6mm_P2.50mm -> Capacitor_THT:C_Disc_D5.0mm_W2.5mm_P2.50mm
- C106: value 47p -> 1000p
- C107: value 0.1u -> 1000p; footprint Capacitor_THT:C_Disc_D5.0mm_W2.5mm_P2.50mm -> Capacitor_THT:C_Disc_D3.0mm_W1.6mm_P2.50mm
- C108, C111: value 120p -> 0.1u; footprint Capacitor_THT:C_Disc_D5.0mm_W2.5mm_P5.00mm -> Capacitor_THT:C_Disc_D5.0mm_W2.5mm_P2.50mm
- C109: value 220p -> 0.01u; footprint Capacitor_THT:C_Disc_D5.0mm_W2.5mm_P5.00mm -> Capacitor_THT:C_Disc_D5.0mm_W2.5mm_P2.50mm
- C11: value 10u -> 22p; footprint Capacitor_THT:CP_Radial_D5.0mm_P2.00mm -> Capacitor_THT:C_Disc_D3.0mm_W1.6mm_P2.50mm; symbol Device:C_Polarized -> Device:C
- C110: value 220p -> 0.1u; footprint Capacitor_THT:C_Disc_D5.0mm_W2.5mm_P5.00mm -> Capacitor_THT:C_Disc_D5.0mm_W2.5mm_P2.50mm
- C113: value 4.7p -> 220u; footprint Capacitor_THT:C_Disc_D3.0mm_W1.6mm_P2.50mm -> Capacitor_THT:CP_Radial_D8.0mm_P3.50mm; symbol Device:C -> Device:C_Polarized
- C115: value 1000p -> 47p
- C117: value 0.1u -> 120p; footprint Capacitor_THT:C_Disc_D5.0mm_W2.5mm_P2.50mm -> Capacitor_THT:C_Disc_D5.0mm_W2.5mm_P5.00mm
- C12, C66: value 220p -> 10u; footprint Capacitor_THT:C_Disc_D3.0mm_W1.6mm_P2.50mm -> Capacitor_THT:CP_Radial_D5.0mm_P2.00mm; symbol Device:C -> Device:C_Polarized
- C14: value 10u -> 220p; footprint Capacitor_THT:CP_Radial_D5.0mm_P2.00mm -> Capacitor_THT:C_Disc_D3.0mm_W1.6mm_P2.50mm; symbol Device:C_Polarized -> Device:C
- C15: value 0.1u -> 10u; footprint Capacitor_THT:C_Disc_D5.0mm_W2.5mm_P2.50mm -> Capacitor_THT:CP_Radial_D5.0mm_P2.00mm; symbol Device:C -> Device:C_Polarized
- C19, C49, C65: value 10u -> 0.1u; footprint Capacitor_THT:CP_Radial_D5.0mm_P2.00mm -> Capacitor_THT:C_Disc_D5.0mm_W2.5mm_P2.50mm; symbol Device:C_Polarized -> Device:C
- C21: value 0.01u -> 10u; footprint Capacitor_THT:C_Disc_D5.0mm_W2.5mm_P2.50mm -> Capacitor_THT:CP_Radial_D5.0mm_P2.00mm; symbol Device:C -> Device:C_Polarized
- C22: value 10u -> 0.01u; footprint Capacitor_THT:CP_Radial_D5.0mm_P2.00mm -> Capacitor_THT:C_Disc_D5.0mm_W2.5mm_P2.50mm; symbol Device:C_Polarized -> Device:C
- C23, C44: value 0.01u -> 47p; footprint Capacitor_THT:C_Disc_D5.0mm_W2.5mm_P2.50mm -> Capacitor_THT:C_Disc_D3.0mm_W1.6mm_P2.50mm
- C29: value 470p -> 0.01u; footprint Capacitor_THT:C_Disc_D3.0mm_W1.6mm_P2.50mm -> Capacitor_THT:C_Disc_D5.0mm_W2.5mm_P2.50mm
- C35: value 47p -> 10u; footprint Capacitor_THT:C_Disc_D3.0mm_W1.6mm_P2.50mm -> Capacitor_THT:CP_Radial_D5.0mm_P2.00mm; symbol Device:C -> Device:C_Polarized
- C36: value 0.1u -> 470p; footprint Capacitor_THT:C_Disc_D5.0mm_W2.5mm_P2.50mm -> Capacitor_THT:C_Disc_D3.0mm_W1.6mm_P2.50mm
- C39: value 27p -> 0.1u; footprint Capacitor_THT:C_Disc_D3.0mm_W1.6mm_P2.50mm -> Capacitor_THT:C_Disc_D5.0mm_W2.5mm_P2.50mm
- C42: value 68p -> 0.1u; footprint Capacitor_THT:C_Disc_D3.0mm_W1.6mm_P2.50mm -> Capacitor_THT:C_Disc_D5.0mm_W2.5mm_P2.50mm
- C43: value 220p -> 0.01u; footprint Capacitor_THT:C_Disc_D3.0mm_W1.6mm_P2.50mm -> Capacitor_THT:C_Disc_D5.0mm_W2.5mm_P2.50mm
- C46: value 56p -> 0.1u; footprint Capacitor_THT:C_Disc_D3.0mm_W1.6mm_P2.50mm -> Capacitor_THT:C_Disc_D5.0mm_W2.5mm_P2.50mm
- C48: value 2.2n -> 27p; footprint Capacitor_THT:C_Disc_D5.0mm_W2.5mm_P2.50mm -> Capacitor_THT:C_Disc_D3.0mm_W1.6mm_P2.50mm
- C50: value 0.047u -> 0.1u
- C51: value 1u -> 68p; footprint Capacitor_THT:C_Disc_D5.0mm_W2.5mm_P2.50mm -> Capacitor_THT:C_Disc_D3.0mm_W1.6mm_P2.50mm
- C52, C75: value 0.1u -> 220p; footprint Capacitor_THT:C_Disc_D5.0mm_W2.5mm_P2.50mm -> Capacitor_THT:C_Disc_D3.0mm_W1.6mm_P2.50mm
- C55: value 100u -> 56p; footprint Capacitor_THT:CP_Radial_D6.3mm_P2.50mm -> Capacitor_THT:C_Disc_D3.0mm_W1.6mm_P2.50mm; symbol Device:C_Polarized -> Device:C
- C57: value 10u -> 2.2n; footprint Capacitor_THT:CP_Radial_D5.0mm_P2.00mm -> Capacitor_THT:C_Disc_D5.0mm_W2.5mm_P2.50mm; symbol Device:C_Polarized -> Device:C
- C58: value 0.047u -> 10u; footprint Capacitor_THT:C_Disc_D5.0mm_W2.5mm_P2.50mm -> Capacitor_THT:CP_Radial_D5.0mm_P2.00mm; symbol Device:C -> Device:C_Polarized
- C59: value 0.47u -> 0.047u
- C60: value 220u -> 1u; footprint Capacitor_THT:CP_Radial_D6.3mm_P2.50mm -> Capacitor_THT:C_Disc_D5.0mm_W2.5mm_P2.50mm; symbol Device:C_Polarized -> Device:C
- C61, C63: value 47u -> 0.1u; footprint Capacitor_THT:CP_Radial_D5.0mm_P2.00mm -> Capacitor_THT:C_Disc_D5.0mm_W2.5mm_P2.50mm; symbol Device:C_Polarized -> Device:C
- C62: value 1u -> 0.01u
- C64: value 47u -> 100u; footprint Capacitor_THT:CP_Radial_D5.0mm_P2.00mm -> Capacitor_THT:CP_Radial_D6.3mm_P2.50mm
- C67: value 1u -> 0.047u
- C68: value 0.1u -> 0.47u
- C69: value 2.2n -> 220u; footprint Capacitor_THT:C_Disc_D5.0mm_W2.5mm_P2.50mm -> Capacitor_THT:CP_Radial_D6.3mm_P2.50mm; symbol Device:C -> Device:C_Polarized
- C70: value 4.7n -> 47u; footprint Capacitor_THT:C_Disc_D5.0mm_W2.5mm_P2.50mm -> Capacitor_THT:CP_Radial_D5.0mm_P2.00mm; symbol Device:C -> Device:C_Polarized
- C71: value 68p -> 1u; footprint Capacitor_THT:C_Disc_D3.0mm_W1.6mm_P2.50mm -> Capacitor_THT:C_Disc_D5.0mm_W2.5mm_P2.50mm
- C72: value 1u -> 47u; footprint Capacitor_THT:C_Disc_D5.0mm_W2.5mm_P2.50mm -> Capacitor_THT:CP_Radial_D5.0mm_P2.00mm; symbol Device:C -> Device:C_Polarized
- C73: value 0.1u -> 47u; footprint Capacitor_THT:C_Disc_D5.0mm_W2.5mm_P2.50mm -> Capacitor_THT:CP_Radial_D5.0mm_P2.00mm; symbol Device:C -> Device:C_Polarized
- C76: value 100p -> 1u; footprint Capacitor_THT:C_Disc_D3.0mm_W1.6mm_P2.50mm -> Capacitor_THT:C_Disc_D5.0mm_W2.5mm_P2.50mm
- C78: value 0.1u -> 2.2n
- C79: value 22p -> 4.7n; footprint Capacitor_THT:C_Disc_D3.0mm_W1.6mm_P2.50mm -> Capacitor_THT:C_Disc_D5.0mm_W2.5mm_P2.50mm
- C8: value 2p -> 0.01u; footprint Capacitor_THT:C_Disc_D3.0mm_W1.6mm_P2.50mm -> Capacitor_THT:C_Disc_D5.0mm_W2.5mm_P2.50mm
- C80: value 1p -> 68p
- C81: value 22p -> 1u; footprint Capacitor_THT:C_Disc_D3.0mm_W1.6mm_P2.50mm -> Capacitor_THT:C_Disc_D5.0mm_W2.5mm_P2.50mm
- C83: value 100p -> 10u; footprint Capacitor_THT:C_Disc_D3.0mm_W1.6mm_P2.50mm -> Capacitor_THT:CP_Radial_D5.0mm_P2.00mm; symbol Device:C -> Device:C_Polarized
- C84: value 82p -> 0.1u; footprint Capacitor_THT:C_Disc_D3.0mm_W1.6mm_P2.50mm -> Capacitor_THT:C_Disc_D5.0mm_W2.5mm_P2.50mm
- C85, C92: value 0.01u -> 100p; footprint Capacitor_THT:C_Disc_D5.0mm_W2.5mm_P2.50mm -> Capacitor_THT:C_Disc_D3.0mm_W1.6mm_P2.50mm
- C88, C90: value 0.01u -> 22p; footprint Capacitor_THT:C_Disc_D5.0mm_W2.5mm_P2.50mm -> Capacitor_THT:C_Disc_D3.0mm_W1.6mm_P2.50mm
- C89: value 0.1u -> 1p; footprint Capacitor_THT:C_Disc_D5.0mm_W2.5mm_P2.50mm -> Capacitor_THT:C_Disc_D3.0mm_W1.6mm_P2.50mm
- C9: value 0.1u -> 2p; footprint Capacitor_THT:C_Disc_D5.0mm_W2.5mm_P2.50mm -> Capacitor_THT:C_Disc_D3.0mm_W1.6mm_P2.50mm
- C93: value 0.1u -> 82p; footprint Capacitor_THT:C_Disc_D5.0mm_W2.5mm_P2.50mm -> Capacitor_THT:C_Disc_D3.0mm_W1.6mm_P2.50mm
- C94: value 180p -> 0.01u; footprint Capacitor_THT:C_Disc_D3.0mm_W1.6mm_P2.50mm -> Capacitor_THT:C_Disc_D5.0mm_W2.5mm_P2.50mm
- C95: value 120p -> 0.01u; footprint Capacitor_THT:C_Disc_D3.0mm_W1.6mm_P2.50mm -> Capacitor_THT:C_Disc_D5.0mm_W2.5mm_P2.50mm
- C97: value 1000p -> 0.01u; footprint Capacitor_THT:C_Disc_D3.0mm_W1.6mm_P2.50mm -> Capacitor_THT:C_Disc_D5.0mm_W2.5mm_P2.50mm
- C98: value 1000p -> 0.1u; footprint Capacitor_THT:C_Disc_D3.0mm_W1.6mm_P2.50mm -> Capacitor_THT:C_Disc_D5.0mm_W2.5mm_P2.50mm
- L10: value 10uH -> FT37-43 10T; footprint Inductor_THT:L_Axial_L9.5mm_D4.0mm_P2.54mm_Vertical_Fastron_SMCC -> Serrasoid_TRX:L_T50_2pin_Vertical
- L11: value 1uH -> 10uH
- L12: value FT50-43 8T -> 1uH; footprint Serrasoid_TRX:L_T50_2pin_Vertical -> Inductor_THT:L_Axial_L9.5mm_D4.0mm_P2.54mm_Vertical_Fastron_SMCC
- L13: value T50-6 9T -> FT50-43 8T
- L14: value T50-6 10T -> T50-6 9T
- L15: value T50-6 9T -> T50-6 10T
- L16: value 4.7uH -> T50-6 9T; footprint Inductor_THT:L_Axial_L9.5mm_D4.0mm_P2.54mm_Vertical_Fastron_SMCC -> Serrasoid_TRX:L_T50_2pin_Vertical
- L3: value T30-6 17T/2T -> 4.7uH; footprint Serrasoid_TRX:L_T30_3pin_Vertical -> Inductor_THT:L_Axial_L9.5mm_D4.0mm_P2.54mm_Vertical_Fastron_SMCC; symbol Serrasoid_TRX:L_Tap -> Device:L
- L4, L8: value 10uH -> T30-6 17T/2T; footprint Inductor_THT:L_Axial_L9.5mm_D4.0mm_P2.54mm_Vertical_Fastron_SMCC -> Serrasoid_TRX:L_T30_3pin_Vertical; symbol Device:L -> Serrasoid_TRX:L_Tap
- L5: value T50-6 15T -> 10uH; footprint Serrasoid_TRX:L_T50_2pin_Vertical -> Inductor_THT:L_Axial_L9.5mm_D4.0mm_P2.54mm_Vertical_Fastron_SMCC
- L6: value T30-6 17T/2T -> T50-6 15T; footprint Serrasoid_TRX:L_T30_3pin_Vertical -> Serrasoid_TRX:L_T50_2pin_Vertical; symbol Serrasoid_TRX:L_Tap -> Device:L
- L9: value FT37-43 10T -> 10uH; footprint Serrasoid_TRX:L_T50_2pin_Vertical -> Inductor_THT:L_Axial_L9.5mm_D4.0mm_P2.54mm_Vertical_Fastron_SMCC
- Q1: value 2N3819 -> 2SC1815; symbol Transistor_FET:2N3819 -> Transistor_BJT:Q_NPN_ECB
- Q10: value RD16HHF1 -> RD06HHF1
- Q2: value 2SC1815 -> 2N3819; symbol Transistor_BJT:Q_NPN_ECB -> Transistor_FET:2N3819
- Q6: value 2N7000 -> 2SC1815; symbol Transistor_FET:2N7000 -> Transistor_BJT:Q_NPN_ECB
- Q7: value 2SA1015 -> 2N7000; symbol Transistor_BJT:Q_PNP_ECB -> Transistor_FET:2N7000
- Q8: value 2N3866 -> 2SA1015; footprint Package_TO_SOT_THT:TO-39-3 -> Package_TO_SOT_THT:TO-92_Inline; symbol Transistor_BJT:Q_NPN_EBC -> Transistor_BJT:Q_PNP_ECB
- Q9: value RD06HHF1 -> 2N3866; footprint Package_TO_SOT_THT:TO-220-3_Vertical -> Package_TO_SOT_THT:TO-39-3; symbol Serrasoid_TRX:RD_MOSFET_GSD -> Transistor_BJT:Q_NPN_EBC
- R1: value 5.6k -> 2.2k
- R10: value 1.5k -> 4.7k
- R11: value 100 -> 1.5k
- R12, R44: value 1k -> 330
- R13: value 22k -> 1.2k
- R15: value 22k -> 1.5k
- R16: value 4.7k -> 100
- R17: value 1.5k -> 10
- R18: value 82 -> 1k
- R19: value 180 -> 22k
- R20, R27: value 10k -> 1k
- R21: value 1k -> 22k
- R22, R32, R34, R41: value 10k -> 4.7k
- R23: value 10k -> 1.5k
- R24: value 1M -> 82
- R25: value 20k -> 180
- R26, R28, R35: value 4.7k -> 10k
- R30: value 220 -> 1M
- R31: value 10k -> 20k
- R36: value 10k -> 220
- R37, R38, R39: value 330 -> 10k
- R4: value 5.6k -> 22k
- R40: value 470k -> 10k
- R43: value 10 -> 330
- R45: value 100k -> 330
- R46: value 10k -> 470k
- R48: value 22k -> 10k
- R49, R79: value 470 -> 10
- R50: value 2.2k -> 1k
- R51: value 10k -> 100k
- R53: value 1.5k -> 10k
- R54: value 10k -> 22k
- R55: value 220k -> 470
- R56: value 10k -> 2.2k
- R57: value 100k -> 10k
- R58, R62: value 100 -> 10k
- R59: value 2.2k -> 1.5k
- R6: value 1.5k -> 27
- R60: value 15k -> 10k
- R61: value 15k -> 220k
- R63: value 1.5k -> 100k
- R64: value 10k -> 100
- R65: value 100k -> 2.2k
- R66: value 10k -> 15k
- R67: value 2.2k -> 15k
- R68: value 120 -> 100
- R69: value 1.8k -> 1.5k
- R7: value 330 -> 220
- R70: value 510 -> 10k
- R71: value 560 -> 100k
- R72: value 4.7 -> 10k
- R73: value 10 -> 2.2k
- R74: value 47 -> 120
- R75: value 10 -> 1.8k
- R76: value 1k -> 510
- R77: value 3.3k -> 560
- R78: value 1k -> 4.7
- R8: value 1.2k -> 5.6k
- R80: value 100 -> 47; footprint Resistor_THT:R_Axial_DIN0414_L11.9mm_D4.5mm_P5.08mm_Vertical -> Resistor_THT:R_Axial_DIN0207_L6.3mm_D2.5mm_P2.54mm_Vertical
- R81: value 100 -> 10; footprint Resistor_THT:R_Axial_DIN0414_L11.9mm_D4.5mm_P5.08mm_Vertical -> Resistor_THT:R_Axial_DIN0207_L6.3mm_D2.5mm_P2.54mm_Vertical
- R83: value 10 -> 3.3k
- R84: value 1M -> 1k
- R85: value 1M -> 470
- R86: value 3.3k -> 100; footprint Resistor_THT:R_Axial_DIN0207_L6.3mm_D2.5mm_P2.54mm_Vertical -> Resistor_THT:R_Axial_DIN0414_L11.9mm_D4.5mm_P5.08mm_Vertical
- R87: value 910 -> 100; footprint Resistor_THT:R_Axial_DIN0207_L6.3mm_D2.5mm_P2.54mm_Vertical -> Resistor_THT:R_Axial_DIN0414_L11.9mm_D4.5mm_P5.08mm_Vertical
- R88: value 330 -> 1k
- R89: value 1k -> 10
- R9: value 1k -> 5.6k
- R90: value 10k -> 1M
- R92: value 47k -> 3.3k
- R93: value 10k -> 910
- U10: value AE-Si5351A -> NJM2594V; footprint Serrasoid_TRX:DIP-8_W7.62mm -> Package_SO:TSSOP-8_4.4x3mm_P0.65mm; symbol Serrasoid_TRX:Si5351_Module -> Serrasoid_TRX:NJM2594
- U11: value 74HCU04 -> AE-Si5351A; footprint Package_DIP:DIP-14_W7.62mm_Socket -> Serrasoid_TRX:DIP-8_W7.62mm; symbol 74xx:74HC04 -> Serrasoid_TRX:Si5351_Module
- U12: value MC3361 -> 74HCU04; footprint Package_DIP:DIP-16_W7.62mm_Socket -> Package_DIP:DIP-14_W7.62mm_Socket; symbol Serrasoid_TRX:MC3361 -> 74xx:74HC04
- U13: value XIAO ESP32C3 -> ADS1115 module; footprint Serrasoid_TRX:Seeeduino_XIAO_Socket -> Serrasoid_TRX:ADS1115_Module_Socket; symbol Serrasoid_TRX:XIAO_ESP32C3 -> Serrasoid_TRX:ADS1115_Module
- U14: value MCP6002 -> MC3361; footprint Package_DIP:DIP-8_W7.62mm_Socket -> Package_DIP:DIP-16_W7.62mm_Socket; symbol Amplifier_Operational:MCP6002-xP -> Serrasoid_TRX:MC3361
- U15: value LM386N-1 -> XIAO ESP32C3; footprint Package_DIP:DIP-8_W7.62mm_Socket -> Serrasoid_TRX:Seeeduino_XIAO_Socket; symbol Amplifier_Audio:LM386 -> Serrasoid_TRX:XIAO_ESP32C3
- U16: value MCP6004 -> MCP6002; footprint Package_DIP:DIP-14_W7.62mm_Socket -> Package_DIP:DIP-8_W7.62mm_Socket; symbol Amplifier_Operational:MCP6004 -> Amplifier_Operational:MCP6002-xP
- U17: value 74HCT4017 -> LM386N-1; footprint Package_DIP:DIP-16_W7.62mm_Socket -> Package_DIP:DIP-8_W7.62mm_Socket; symbol 4xxx:4017 -> Amplifier_Audio:LM386
- U18: value MAX913CPA -> MCP6004; footprint Package_DIP:DIP-8_W7.62mm_Socket -> Package_DIP:DIP-14_W7.62mm_Socket; symbol Comparator:LT1016 -> Amplifier_Operational:MCP6004
- U19: value 74HCT123 -> 74HCT4017; symbol 74xx:74HC123 -> 4xxx:4017
- U20: value 74AC14 -> MAX913CPA; footprint Package_DIP:DIP-14_W7.62mm_Socket -> Package_DIP:DIP-8_W7.62mm_Socket; symbol 74xx:74HC14 -> Comparator:LT1016
- U21: value 74AC86 -> 74HCT123; footprint Package_DIP:DIP-14_W7.62mm_Socket -> Package_DIP:DIP-16_W7.62mm_Socket; symbol 74xx:74HC86 -> 74xx:74HC123
- U22: value 74HCU04 -> 74AC14; symbol 74xx:74HC04 -> 74xx:74HC14
- U23: value 74AC14 -> 74AC86; symbol 74xx:74HC14 -> 74xx:74HC86
- U9: value NJM2594V -> AD8307ANZ; footprint Package_SO:TSSOP-8_4.4x3mm_P0.65mm -> Package_DIP:DIP-8_W7.62mm_Socket; symbol Serrasoid_TRX:NJM2594 -> Serrasoid_TRX:AD8307
Connections:
- net +13V8: now also C100.1, C110.1, C112.1, C113.1, L10.1, L13.1; no longer C101.1, C103.1, C104.1, C91.1, L12.1, L9.1
- net +3V3S: now also C35.1, C37.1, U11.1 (VDDO), U11.8 (VDD); no longer C28.1, C30.1, U10.1 (VDDO), U10.8 (VDD)
- net +3V3X: now also R32.1, R34.1, R35.1, R47.1, R48.1, U13.1 (VDD), U15.10 (3V3); no longer R23.1, R26.1, R28.1, R41.1, R42.1, U13.10 (3V3)
- net +5V: now also C21.1, C24.1; no longer C19.1, C20.1
- net +5VA: now also C41.1, C49.2, C50.2, C52.2, C65.1, R17.1, R31.2, R38.1, U10.1 (V+), U14.4 (VCC), U16.8 (V+); no longer C32.1, C40.2, C41.2, C43.2, C47.1, R25.2, R32.1, U12.4 (VCC), U9.1 (V+)
- net +5VT: now also C10.1, C102.1, C108.1, C116.1, C16.1, C28.1, C34.1, C39.1, C82.1, C84.1, C86.1, C87.1, C98.1, R55.1, R57.1, R69.1, R73.1, U19.16 (VDD), U20.1 (V+), U21.16 (VCC), U21.3 (Clr), U21.9 (A), U23.14 (VCC), U12.14 (VCC), U18.4 (V+), U24.14 (VCC), U25.14 (VCC); no longer C107.1, C15.1, C22.1, C27.1, C31.1, C68.1, C73.1, C75.1, C78.1, C89.1, C9.1, C93.1, C99.1, R49.1, R51.1, R63.1, R67.1, U17.16 (VDD), U18.1 (V+), U19.3 (Clr)
- net +8V: now also C15.1, C19.1; no longer C14.1, C16.1
- net GND: now also C102.2, C113.2, C115.2, C21.2, C34.2, C35.2, C38.2, C40.2, C41.2, C42.2, C45.2, C48.2, C53.2, C66.2, C67.2, C70.2, C72.2, C73.2, C80.2, C87.2, C92.2, C97.2, C98.2, L12.2, L4.3, L8.3, Q7.1 (S), R10.2, R12.2, R20.2, R25.2, R28.2, R33.2, R42.2, R51.2, R54.2, R58.2, R70.2, R74.2, R79.2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; no longer C101.2, C106.2, C107.2, C111.2, C32.2, C33.2, C44.2, C47.2, C49.2, C50.2, C52.2, C57.2, C63.2, C71.2, C75.2, C78.2, C79.2, C81.2, C85.2, C89.2, C9.2, C91.2, C96.2, L10.2, L16.2, L3.3, L6.3, Q3.1 (E), Q9.2 (S), R11.2, R14.2, R19.2, R27.2, R36.2, R45.2, R46.2, R48.2, R64.2, R68.2, R73.2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
- net RX8V: now also C22.1, C31.1, C45.1, C61.1, C64.1, C72.1, L3.1, L5.1, R14.1, R21.1, R23.1, R26.1, R4.1, U17.6 (V+); no longer C24.1, C36.1, C52.1, C55.1, C63.1, L4.1, R15.1, R17.1, R20.1, R9.1, U15.6 (V+)
- net TX8V: now also C73.1, C95.1, L9.1, R59.1, R83.1, R92.1; no longer C64.1, C86.1, L8.1, R53.1, R71.1, R86.1
- net at TP4.1: now also U20.3 (-), U18.13 (-), U18.14; no longer U18.3 (-)
- net at D6.1 (K), D7.2 (A): now also C63.2; no longer C54.2
- net at R67.2: now also C78.1, U18.10 (+); no longer VR5.1
- net at R87.1: now also C101.2, R86.1, R88.2, R89.1; no longer U21.4
- net at U21.6 (Cext): no longer R89.1
- net at C13.1, R2.2: now also R8.1; no longer R4.1
- net at L6.2: now also C44.1, C48.1, Q4.2 (C), R30.1, TC3.1, U12.1; no longer C53.2
- net at VR3.1: now also C81.2; no longer C72.2
- net at VR3.2: now also R71.1; no longer R65.1
- net at VR2.1: now also R69.2; no longer R63.2
- net at VR2.2, VR2.3: now also Q8.1 (E); no longer Q7.1 (E)
- net at D8.2 (A), K1.16: now also Q6.2 (C); no longer Q5.2 (C)
- net at C105.1, R87.2: now also R86.2
- net at VR1.1: now also C76.2; no longer C67.2
- net at C40.1: now also U13.7 (A0), U9.4 (OUT); no longer U12.6 (DEC1)
- net at FL2.1 (IN): now also U14.3 (MIX_OUT); no longer U12.3 (MIX_OUT)
- net at FL2.3 (OUT): now also U14.5 (LIM_IN); no longer U12.5 (LIM_IN)
- net at C60.2: now also J4.1 (Pin_1); no longer J6.1 (Pin_1)
- net at L9.2, Q9.3 (C): now also C96.1; no longer C92.1
- net at L7.2 (TAP): now also C62.2; no longer C82.1
- net at Q3.3 (B), R22.1: now also C43.2, R21.2; no longer R20.2
- net at D10.1 (K), D9.2 (A): now also R65.2, R66.1; no longer R59.2, R60.1
- net at Q10.1 (G): now also R81.2; no longer R83.2
- net at C94.1, R78.2: now also R79.1; no longer C97.1, L10.1
- net at R44.1: now also U12.8; no longer U13.11 (D10/MOSI)
- net at J3.2 (Pin_2): now also U15.7 (D6/TX); no longer U13.7 (D6/TX)
- net at U13.8 (A1): no longer D5.1 (K)
- net at J7.2 (Pin_2): now also R27.1; no longer R21.1
- net at C88.1: now also C89.1, L7.1, TC4.1; no longer R74.2
- net at U23.4: now also R93.1, U22.10
- net at R72.1: now also C83.1, VR4.2; no longer Q8.1 (E)
- net at U22.4: now also U23.5; no longer R91.2
- net at R62.2: now also C74.1, C78.2, D10.2 (A), D9.1 (K), R57.2, R58.1, U18.3 (+), VR1.3, VR3.3; no longer Q6.2 (G)
- net at T1.1 (AA): now also C111.2; no longer C102.2
- net at R66.2: now also C79.1, R67.1; no longer R65.2
- net at U10.5 (SIG): now also C32.2; no longer R58.1
- net at R70.1: now also C82.2, D12.1 (K), Q8.3 (B); no longer U21.9
- net at R54.1: now also R53.2, U15.3 (D2/A2); no longer C62.2
- net at FL1.1 (IN): now also C47.2; no longer C38.2
- net at FL1.3 (OUT): now also R1.1, U14.16 (MIX_IN); no longer U12.16 (MIX_IN)
- net at R60.2, R61.1: now also C75.1, U18.2 (-); no longer C70.1
- net at R43.2: now also C62.1, R44.2, R45.2; no longer C58.1
- net at R80.1, R81.1, R82.2: now also C96.2; no longer C92.2, R83.1
- net at C33.1: now also R13.2, R16.1; no longer U9.6 (BYP)
- net at C76.1: now also C75.2, R61.2, U18.1; no longer U19.14 (Cext)
- net at VR5.2, VR5.3: now also C85.2, U21.15 (RCext); no longer C76.2, U19.15 (RCext)
- net at R18.2, R19.1: now also C36.1, TP1.1; no longer C37.1
- net at TP6.1, U1.3 (C): now also U23.11
- net at R88.1: now also C109.1, VR7.2; no longer U23.2
- net at R18.1: now also R15.1, U7.1; no longer Q2.1 (E)
- net at C38.1, R17.2: now also U9.6 (ENB), U9.7 (VPS); no longer Q2.2 (C)
- net at J4.2 (Pin_2): now also R41.1; no longer R35.1
- net at C106.1: now also C103.1, L11.1, R84.2; no longer R88.2
- net at L14.2, L15.1: now also C118.1; no longer C110.1
- net at R75.2: now also C92.1, U22.1; no longer Q9.1 (G)
- net at C18.1, R6.2: now also R7.1
- net at TP2.1: now also R43.1, U12.6; no longer R37.1
- net at R33.1: now also C58.1, R38.2, U16.3 (+), U16.5 (+); no longer C48.2
- net at U1.5 (Q), U3.1: now also R2.1; no longer R1.1
- net at U1.9 (Q), U3.2: now also R3.1; no longer R2.1
- net at VR1.2: now also U18.5 (+); no longer U16.5 (+)
- net at J9.1 (Pin_1): now also R59.2; no longer R53.2
- net at C4.1, L1.1, TC1.1: now also C9.1; no longer C8.1
- net at C51.2: now also C52.1, U14.2 (OSC_E); no longer J4.1 (Pin_1)
- net at VR7.1: now also R92.2; no longer R86.2
- net at U17.3 (+): now also Q5.2 (C), R41.2; no longer R62.1
- net at R39.1: now also C57.2
- net at U17.5: now also C69.1, R49.1
- net at U17.7 (BYPASS): now also C66.1
- net at R11.1, R8.2: now also U7.3 (+); no longer C26.1
- net at L3.2: now also C23.1, C26.1, Q1.2 (C)
- net at U10.6 (BYP): now also C42.1; no longer R8.1
- net at U10.7 (CARR): now also C33.2
- net at U22.2: now also U23.2; no longer R84.2
- net at U20.2 (+): now also C80.1, Q7.3 (D), Q8.2 (C), TP3.1; no longer U21.2
- net at U15.1 (D0/A0): now also C53.1, R27.2, R35.2
- net at C57.1: now also R37.1, U14.9 (AUDIO); no longer U15.7 (BYPASS)
- net at U15.8 (VIN): now also D5.1 (K)
- net at C26.2: now also U9.8 (INP); no longer U9.7 (CARR)
- net at U22.8: now also U23.13
- net at U22.12: now also R76.1, U23.9
- net at R78.1: now also Q9.1 (E); no longer U21.3
- net at U19.2 (Q1): no longer U18.7 (Q)
- net at U1.11 (C): now also U12.4
- net at L2.2, U5.1 (IN): now also C12.1; no longer C11.1
- net at C25.2: now also R9.2, U7.2 (-); no longer U9.5 (SIG)
- net at R77.2: now also C91.2, Q9.2 (B), R74.1; no longer VR6.1
- new net: C54.1, C55.1, R36.2
- new net: C47.1, Q3.2 (C), R23.2
- new net: U22.6, U23.10
- new net: R85.1, U23.8
- new net: R31.1, U14.8 (QUAD), X2.1
- new net: C89.2, C90.1, L8.1, TC5.1
- new net: C91.1, L8.2 (TAP)
- new net: C67.1, R49.2
- new net: C11.1, C9.2, L4.1, Q2.2 (G), R10.1, TC2.1
- new net: J2.2 (Pin_2), R34.2, U11.2 (SCL), U13.3 (SCL), U15.6 (D5/SCL)
- new net: J2.3 (Pin_3), R32.2, U11.3 (SDA), U13.4 (SDA), U15.5 (D4/SDA)
- new net: R30.2, R36.1, U12.11, U12.2, U12.3, U12.5, U12.9
- new net: C59.1, C60.1, R37.2
- new net: C120.1, C122.1, K1.8, L16.2
- new net: C70.1, R55.2, R56.1
- new net: C71.1, J7.1 (Pin_1), R56.2
- new net: C106.2, R90.1, U24.1
- new net: R90.2, U22.11, U24.2
- new net: C85.1, U21.14 (Cext)
- new net: C68.1, D7.1 (K), R51.1, R53.1
- new net: Q3.1 (E), R24.1
- new net: R71.2, R72.2, U18.12 (+)
- new net: C101.1, L10.2, Q10.3 (D)
- new net: C50.1, U14.7 (DEC2)
- new net: C97.1, R80.2
- new net: C124.2, R97.1, U24.3
- new net: R97.2, U22.13, U24.4
- new net: C25.1, R15.2
- new net: R13.1, U11.6 (CLK1)
- new net: C29.1, Q2.3 (S), R12.1
- new net: R95.1, U23.6
- new net: C79.2, C81.1, U18.8, U18.9 (-)
- new net: C107.2, R91.1, U24.5
- new net: R91.2, U24.6, U25.1
- new net: Q6.3 (B), R50.2, R52.1
- new net: C46.1, R24.2, R25.1
- new net: C117.1, L14.1, T1.3 (SA)
- new net: C63.1, R46.2, U16.1
- new net: C69.2, J6.1 (Pin_1)
- new net: C27.1, U9.1 (INM)
- new net: C99.1, R82.1, VR6.2
- new net: R75.1, TP5.1, U21.13 (Q), U23.1
- new net: C8.2, Q1.3 (B), R4.2, R5.1
- new net: Q4.3 (B), R26.2, R28.1
- new net: C111.1, L13.2, Q11.3 (D)
- new net: C71.2, R60.1
- new net: R83.2, VR6.1
- new net: R39.2, R46.1, U16.2 (-)
- new net: R73.2, VR5.1
- new net: R94.1, U23.12, U25.2
- new net: J5.3 (Pin_3), R48.2, U15.12 (D9/MISO)
- new net: R50.1, U15.11 (D10/MOSI)
- new net: Q7.2 (G), R68.2
- new net: C32.1, L5.2, Q2.1 (D), R14.2
- new net: C119.1, L15.2, L16.1
- new net: C44.2, D4.1 (K), R19.2
- new net: R68.1, U19.3 (Q0)
- new net: C54.2, L6.1
- new net: C122.2, C123.1, D13.2 (A), R96.1
- new net: C121.1, C124.1, L17.1, R95.2
- new net: R40.1, U15.14 (D7/RX)
- new net: Q5.3 (B), R40.2, R42.1
- new net: C20.1, R11.2
- new net: C51.1, U14.1 (OSC_B), X1.1
- new net: C93.1, R76.2, U22.5
- new net: C14.1, R3.2, R9.1
- new net: U16.6 (-), U16.7
- new net: C30.1, U9.3 (OFS)
- new net: R45.1, U12.10
- new net: Q11.1 (G), R89.2
- new net: R62.1, R63.1, U18.6 (-)
- new net: C125.1, D13.1 (K), R98.1, R99.1
- new net: C104.1, C107.1, L12.1, R85.2
- new net: R84.1, U23.3
- new net: C126.1, R99.2, U15.2 (D1/A1)
- new net: J5.2 (Pin_2), R47.2, U15.13 (D8/SCK)
- new net: C43.1, R20.1, U10.3 (OUT2)
- new net: U20.7 (Q), U21.2 (B)
- new net: J5.1 (Pin_1), R29.2, U15.4 (D3/A3)
- new net: C8.1, R1.2
- new net: C49.1, U14.6 (DEC1)
- new net: R64.1, U11.5 (CLK0)
- new net: C115.1, R94.2, U22.9
- new net: C114.1, R93.2, U22.3
- new net: Q1.1 (E), R6.1
- new net: R64.2, U19.14 (CLK)
- new net: R63.2, R65.1, U18.7
- now unconnected: L4.2, U10.2 (SCL), U13.6 (D5/SCL)
- no-connect marks 42 -> 47
Other:
- moved on the sheet: C10, C100, C101, C102, C103, C105, C106, C107, C108, C109, C110, C111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

Commit message: クレジットを変更
Co-Authored-By: Claude Opus 5.5 <noreply@anthropic.com>
Other:
- company: JA6FUF -> 設計 真城和一（JA6FUF/JH1XHX）

Commit message: 入手しにくい部品を置き換え（74HCT4017・MAX913・2N3866）
- 74HCT4017（製造中止）: 外して、Si5351 の CLK0 を 1.83125MHz（送信周波数 ÷ 16）に。リセットパルスは
  74HCT123 の 2 回路目（CLK0 の立ち上がり、22p・1.5k で約 50〜100ns）で作る。スケッチも ÷16 に変更
- MAX913（入手難）: 2SA1015 2 個の差動対（電流 約 2.3mA、負荷 1k）に。COMP_N の立ち下がりで 74HCT123 の 1 回路目をトリガ
- 2N3866（製造中止）: 2N2222A（TO-92）に。エミッタ帰還 4.7Ω ＋ 18Ω で約 33mA
- 基板を配置・配線し直し（極小配線の重なりによるショートを除去して引き直し）: DRC エラー 0・未接続 0・食い違い 0、
  ERC 0・照合 875 ピン一致。ガーバー・3D 画像・部品実装図・A3 配置図・回路図 PDF・docx・図を作り直し
- 購入用部品表（2N2222A・18Ω を追加、74HCT123 は DigiKey 在庫あり、要確認 8 行）、README、回路図論理チェック・基板チェックの追補、
  ケースの部品位置（干渉チェック通過、形は変わらず）

Co-Authored-By: Claude Opus 5.5 <noreply@anthropic.com>
Parts:
- removed C126: 0.1u, Capacitor_THT:C_Disc_D5.0mm_W2.5mm_P2.50mm, symbol Device:C
- removed U24: 74HCU04, Package_DIP:DIP-14_W7.62mm_Socket, symbol 74xx:74HC04
- removed U25: 74AC14, Package_DIP:DIP-14_W7.62mm_Socket, symbol 74xx:74HC14
- added Q12: RD06HHF1, Package_TO_SOT_THT:TO-220-3_Vertical, symbol Serrasoid_TRX:RD_MOSFET_GSD
- added Q13: RD16HHF1, Package_TO_SOT_THT:TO-220-3_Vertical, symbol Serrasoid_TRX:RD_MOSFET_GSD
- added R100: 1M, Resistor_THT:R_Axial_DIN0207_L6.3mm_D2.5mm_P2.54mm_Vertical, symbol Device:R
- added R101: 47k, Resistor_THT:R_Axial_DIN0207_L6.3mm_D2.5mm_P2.54mm_Vertical, symbol Device:R
- added R102: 10k, Resistor_THT:R_Axial_DIN0207_L6.3mm_D2.5mm_P2.54mm_Vertical, symbol Device:R
- added TP7: X16, TestPoint:TestPoint_THTPad_D1.5mm_Drill0.7mm, symbol Connector:TestPoint
- added unit 2 of U19
- added unit 3 of U19
- added unit 4 of U20
- added unit 3 of U20
- added unit 6 of U20
- added unit 7 of U20
- added unit 2 of U20
- added unit 5 of U20
- added unit 4 of U21
- added unit 5 of U21
- added unit 7 of U23
- added unit 6 of U23
- C100, C108, C111, C98: value 0.1u -> 0.01u
- C101, C109, C125, C97, C99: value 0.01u -> 0.1u
- C102: value 0.1u -> 180p; footprint Capacitor_THT:C_Disc_D5.0mm_W2.5mm_P2.50mm -> Capacitor_THT:C_Disc_D3.0mm_W1.6mm_P2.50mm
- C103: value 180p -> 120p
- C104: value 120p -> 0.01u; footprint Capacitor_THT:C_Disc_D3.0mm_W1.6mm_P2.50mm -> Capacitor_THT:C_Disc_D5.0mm_W2.5mm_P2.50mm
- C105: value 0.01u -> 1000p; footprint Capacitor_THT:C_Disc_D5.0mm_W2.5mm_P2.50mm -> Capacitor_THT:C_Disc_D3.0mm_W1.6mm_P2.50mm
- C107: value 1000p -> 0.1u; footprint Capacitor_THT:C_Disc_D3.0mm_W1.6mm_P2.50mm -> Capacitor_THT:C_Disc_D5.0mm_W2.5mm_P2.50mm
- C112: value 0.01u -> 220u; footprint Capacitor_THT:C_Disc_D5.0mm_W2.5mm_P2.50mm -> Capacitor_THT:CP_Radial_D8.0mm_P3.50mm; symbol Device:C -> Device:C_Polarized
- C113: value 220u -> 100p; footprint Capacitor_THT:CP_Radial_D8.0mm_P3.50mm -> Capacitor_THT:C_Disc_D3.0mm_W1.6mm_P2.50mm; symbol Device:C_Polarized -> Device:C
- C114: value 100p -> 47p
- C115: value 47p -> 0.1u; footprint Capacitor_THT:C_Disc_D3.0mm_W1.6mm_P2.50mm -> Capacitor_THT:C_Disc_D5.0mm_W2.5mm_P2.50mm
- C116: value 0.1u -> 120p; footprint Capacitor_THT:C_Disc_D5.0mm_W2.5mm_P2.50mm -> Capacitor_THT:C_Disc_D5.0mm_W2.5mm_P5.00mm
- C117: value 120p -> 220p
- C119: value 220p -> 120p
- C120: value 120p -> 100p; footprint Capacitor_THT:C_Disc_D5.0mm_W2.5mm_P5.00mm -> Capacitor_THT:C_Disc_D3.0mm_W1.6mm_P2.50mm
- C121: value 100p -> 4.7p
- C122: value 4.7p -> 100p
- C123: value 100p -> 1000p
- C124: value 1000p -> 0.01u; footprint Capacitor_THT:C_Disc_D3.0mm_W1.6mm_P2.50mm -> Capacitor_THT:C_Disc_D5.0mm_W2.5mm_P2.50mm
- C77: value 0.1u -> 2.2n
- C78: value 2.2n -> 4.7n
- C79: value 4.7n -> 68p; footprint Capacitor_THT:C_Disc_D5.0mm_W2.5mm_P2.50mm -> Capacitor_THT:C_Disc_D3.0mm_W1.6mm_P2.50mm
- C80: value 68p -> 1u; footprint Capacitor_THT:C_Disc_D3.0mm_W1.6mm_P2.50mm -> Capacitor_THT:C_Disc_D5.0mm_W2.5mm_P2.50mm
- C81: value 1u -> 0.1u
- C82: value 0.1u -> 10u; footprint Capacitor_THT:C_Disc_D5.0mm_W2.5mm_P2.50mm -> Capacitor_THT:CP_Radial_D5.0mm_P2.00mm; symbol Device:C -> Device:C_Polarized
- C83: value 10u -> 100p; footprint Capacitor_THT:CP_Radial_D5.0mm_P2.00mm -> Capacitor_THT:C_Disc_D3.0mm_W1.6mm_P2.50mm; symbol Device:C_Polarized -> Device:C
- C84, C87: value 0.1u -> 22p; footprint Capacitor_THT:C_Disc_D5.0mm_W2.5mm_P2.50mm -> Capacitor_THT:C_Disc_D3.0mm_W1.6mm_P2.50mm
- C85: value 100p -> 0.1u; footprint Capacitor_THT:C_Disc_D3.0mm_W1.6mm_P2.50mm -> Capacitor_THT:C_Disc_D5.0mm_W2.5mm_P2.50mm
- C88: value 22p -> 1p
- C89: value 1p -> 22p
- C90: value 22p -> 0.01u; footprint Capacitor_THT:C_Disc_D3.0mm_W1.6mm_P2.50mm -> Capacitor_THT:C_Disc_D5.0mm_W2.5mm_P2.50mm
- C91: value 0.01u -> 100p; footprint Capacitor_THT:C_Disc_D5.0mm_W2.5mm_P2.50mm -> Capacitor_THT:C_Disc_D3.0mm_W1.6mm_P2.50mm
- C92: value 100p -> 82p
- C93: value 82p -> 0.01u; footprint Capacitor_THT:C_Disc_D3.0mm_W1.6mm_P2.50mm -> Capacitor_THT:C_Disc_D5.0mm_W2.5mm_P2.50mm
- Q10: value RD06HHF1 -> 2SA1015; footprint Package_TO_SOT_THT:TO-220-3_Vertical -> Package_TO_SOT_THT:TO-92_Inline; symbol Serrasoid_TRX:RD_MOSFET_GSD -> Transistor_BJT:Q_PNP_ECB
- Q11: value RD16HHF1 -> 2N2222A; footprint Package_TO_SOT_THT:TO-220-3_Vertical -> Package_TO_SOT_THT:TO-92_Inline; symbol Serrasoid_TRX:RD_MOSFET_GSD -> Transistor_BJT:Q_NPN_EBC
- Q9: value 2N3866 -> 2SA1015; footprint Package_TO_SOT_THT:TO-39-3 -> Package_TO_SOT_THT:TO-92_Inline; symbol Transistor_BJT:Q_NPN_EBC -> Transistor_BJT:Q_PNP_ECB
- R73: value 2.2k -> 1k
- R74: value 120 -> 1.5k
- R75: value 1.8k -> 1.5k
- R76: value 510 -> 2.2k
- R77: value 560 -> 120
- R78: value 4.7 -> 1.8k
- R79: value 10 -> 510
- R80: value 47 -> 560
- R81: value 10 -> 4.7
- R82: value 1k -> 18
- R83: value 3.3k -> 47
- R84: value 1k -> 10
- R85: value 470 -> 1k
- R86: value 100 -> 3.3k; footprint Resistor_THT:R_Axial_DIN0414_L11.9mm_D4.5mm_P5.08mm_Vertical -> Resistor_THT:R_Axial_DIN0207_L6.3mm_D2.5mm_P2.54mm_Vertical
- R87: value 100 -> 1k; footprint Resistor_THT:R_Axial_DIN0414_L11.9mm_D4.5mm_P5.08mm_Vertical -> Resistor_THT:R_Axial_DIN0207_L6.3mm_D2.5mm_P2.54mm_Vertical
- R88: value 1k -> 470
- R89: value 10 -> 100; footprint Resistor_THT:R_Axial_DIN0207_L6.3mm_D2.5mm_P2.54mm_Vertical -> Resistor_THT:R_Axial_DIN0414_L11.9mm_D4.5mm_P5.08mm_Vertical
- R90: value 1M -> 100; footprint Resistor_THT:R_Axial_DIN0207_L6.3mm_D2.5mm_P2.54mm_Vertical -> Resistor_THT:R_Axial_DIN0414_L11.9mm_D4.5mm_P5.08mm_Vertical
- R91: value 1M -> 1k
- R92: value 3.3k -> 10
- R93: value 910 -> 1M
- R94: value 330 -> 1M
- R95: value 1k -> 3.3k
- R96: value 10k -> 910
- R97: value 1M -> 330
- R98: value 47k -> 1k
- TP5: value PM -> COMP
- TP6: value X16 -> PM
- U19: value 74HCT4017 -> 74HCT123; symbol 4xxx:4017 -> 74xx:74HC123
- U20: value MAX913CPA -> 74AC14; footprint Package_DIP:DIP-8_W7.62mm_Socket -> Package_DIP:DIP-14_W7.62mm_Socket; symbol Comparator:LT1016 -> 74xx:74HC14
- U21: value 74HCT123 -> 74AC86; footprint Package_DIP:DIP-16_W7.62mm_Socket -> Package_DIP:DIP-14_W7.62mm_Socket; symbol 74xx:74HC123 -> 74xx:74HC86
- U22: value 74AC14 -> 74HCU04; symbol 74xx:74HC14 -> 74xx:74HC04
- U23: value 74AC86 -> 74AC14; symbol 74xx:74HC86 -> 74xx:74HC14
Connections:
- net +13V8: now also C109.1, C111.1, C99.1; no longer C100.1, C110.1, C113.1
- net +5VT: now also C101.1, C107.1, C115.1, C81.1, C85.1, C97.1, R74.1, R75.1, R76.1, U19.2 (B), U19.3 (Clr), U19.11 (Clr), U19.16 (VCC), U20.14 (VCC), U21.14 (VCC), U23.14 (VCC); no longer C102.1, C108.1, C116.1, C77.1, C82.1, C84.1, C87.1, C98.1, R73.1, U19.16 (VDD), U20.1 (V+), U21.16 (VCC), U21.3 (Clr), U21.9 (A), U23.14 (VCC)
- net GND: now also C101.2, C107.2, C111.2, C122.2, C124.2, C79.2, C82.2, C85.2, C89.2, C91.2, C96.2, R73.2, R77.2, R82.2, R99.2, U22.11, U22.13, U22.9, U23.11, U23.3, U23.5, U23.9, Q12.2 (S), Q13.2 (S), R101.2, U19.8 (GND), U19.9 (A), U20.7 (GND), U21.7 (GND), U23.13, U23.7 (GND); no longer C100.2, C105.2, C110.2, C121.2, C123.2, C77.2, C80.2, C83.2, C84.2, C88.2, C90.2, C95.2, Q11.2 (S), R74.2, R79.2, R96.2, R98.2, U19.13 (CKEN), U19.15 (Reset), U19.8 (VSS), U20.4 (V-), U20.5 (LATCH), U20.6 (GND), U21.1 (A), U21.10 (B), U21.11 (Clr), U21.8 (GND), U23.7 (GND)
- net TX8V: now also C94.1, R80.1, R86.1, R95.1; no longer C95.1, R77.1, R83.1, R92.1
- net at TP4.1, U18.13 (-), U18.14: now also Q10.3 (B); no longer U20.3 (-)
- net at R66.2, R67.1: now also C78.1; no longer C79.1
- net at R67.2, U18.10 (+): now also C77.1; no longer C78.1
- net at C74.1, D10.2 (A), D9.1 (K)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: now also C77.2; no longer C78.2
- net at U21.5: now also U20.4
- net at U21.6: now also R98.1
- net at U22.6: now also R94.2, U23.1; no longer U23.10
- net at R85.1: now also C98.1, VR6.2; no longer U23.8
- net at VR3.1: now also C80.2; no longer C81.2
- net at C105.1, R87.2: now also C102.1, L11.1; no longer R86.2
- net at L8.1, TC5.1: now also C88.2, C89.1; no longer C89.2, C90.1
- net at L8.2 (TAP): now also C90.1; no longer C91.1
- net at K1.8, L16.2: now also C119.1, C121.1; no longer C120.1, C122.1
- net at C88.1, L7.1, TC4.1: now also C87.1; no longer C89.1
- net at R90.1: now also C100.2, R89.1, R91.2, R92.1; no longer C106.2
- net at R90.2: now also C104.1, R89.2; no longer U22.11
- net at VR5.2, VR5.3: now also C83.2, U19.15 (RCext); no longer C85.2, U21.15 (RCext)
- net at Q10.1 (E): now also Q9.1 (E), R74.2; no longer R81.2
- net at R80.2: now also C90.2, Q11.2 (B), R77.1; no longer C97.1
- net at R97.1: now also U23.2, U21.12; no longer C124.2
- net at R97.2: now also C114.1, U20.9; no longer U22.13
- net at U22.4: now also R100.2, U20.13; no longer U23.5
- net at R72.1, VR4.2: now also C82.1; no longer C83.1
- net at U18.8, U18.9 (-): now also C78.2, C80.1; no longer C79.2, C81.1
- net at R91.1: now also C108.1, VR7.2; no longer C107.2
- net at C103.1, C106.1: now also L12.1, R88.2; no longer L11.1, R84.2
- net at T1.1 (AA): now also C110.2; no longer C111.2
- net at L14.1, T1.3 (SA): now also C116.1; no longer C117.1
- net at Q7.3 (D), Q8.2 (C), TP3.1: now also C79.1, Q9.3 (B); no longer C80.1, U20.2 (+)
- net at D12.1 (K), Q8.3 (B), R70.1: now also C81.2; no longer C82.2
- net at R83.2: now also C96.1; no longer VR6.1
- net at VR5.1: now also R76.2; no longer R73.2
- net at R94.1: now also C106.2, U22.5; no longer U23.12
- net at L14.2, L15.1: now also C117.1; no longer C118.1
- net at L15.2, L16.1: now also C118.1; no longer C119.1
- net at R68.1: now also U19.5 (Q); no longer U19.3 (Q0)
- net at Q11.1 (E): now also R81.1; no longer R89.2
- net at VR7.1: now also R95.2; no longer R92.2
- net at U22.2: now also R93.2, U20.11; no longer U23.2
- net at R84.1: now also C95.2, R83.1, R85.2; no longer U23.3
- net at U15.2 (D1/A1): now also C125.1, R102.2; no longer R99.2
- net at R78.1: now also TP6.1, U19.13 (Q), U21.1; no longer Q9.1 (E)
- net at U21.2: now also U20.2; no longer U20.7 (Q)
- net at U22.8: no longer U23.13
- net at U19.1 (A): now also Q9.2 (C), R73.1, TP5.1
- net at R64.2: now also U19.10 (B); no longer U19.14 (CLK)
- new net: R96.1, U20.10, U21.4
- new net: R87.1, U21.3
- new net: TP7.1, U1.3 (C), U21.11
- new net: C84.1, U19.6 (Cext)
- new net: C105.2, R93.1, U22.1
- new net: C95.1, L9.2, Q11.3 (C)
- new net: C124.1, D13.1 (K), R101.1, R102.1
- new net: C91.1, R78.2, U20.1
- new net: C120.1, C123.1, L17.1, R98.2
- new net: C83.1, U19.14 (Cext)
- new net: C110.1, L13.2, Q13.3 (D)
- new net: U20.8, U21.13
- new net: C123.2, R100.1, U22.3
- new net: C92.1, R79.2, U20.5
- new net: R79.1, U20.12, U21.9
- new net: C93.1, R81.2, R82.1
- new net: C100.1, L10.2, Q12.3 (D)
- new net: U20.6, U21.10
- new net: C121.2, C122.1, D13.2 (A), R99.1
- new net: C113.1, R96.2, U20.3
- new net: R88.1, U21.8
- new net: Q13.1 (G), R92.2
- new net: R86.2, VR6.1
- new net: Q12.1 (G), R84.2
- new net OS2_RC: C84.2, R75.2, U19.7 (RCext)
- now unconnected: U22.10, U22.12, U23.4
- no-connect marks 47 -> 33
Other:
- note added: "送信: マイク → 送信音声 → セラゾイド変調（1.83125MHz で PM）→ 逓倍 ×16（段間同調）→ PLL（VCO 29.3MHz）→ 送信RF（10W）→ ANT 受信: ANT → 受信（2N3819 → NJM2594 → 10.7MHz 増幅 → 10.7MHz → MC3361 → LM386）→ SP 制御: XIAO ESP32C3 ＋ Si5351（CLK0 = 変調基準 1.83125MHz、CLK1 = 受信局発 18.6MHz） ブロックの中もブロックの間も線で結線（電源も線。電源の名前は出どころの電源記号で示す。GND だけ GND 記号）"
- note removed: "送信: マイク → 送信音声 → セラゾイド変調（1.83125MHz で PM）→ 逓倍 ×16（段間同調）→ PLL（VCO 29.3MHz）→ 送信RF（10W）→ ANT 受信: ANT → 受信（2N3819 → NJM2594 → 10.7MHz 増幅 → 10.7MHz → MC3361 → LM386）→ SP 制御: XIAO ESP32C3 ＋ Si5351（CLK0 = 変調基準 18.3125MHz、CLK1 = 受信局発 18.6MHz） ブロックの中もブロックの間も線で結線（電源も線。電源の名前は出どころの電源記号で示す。GND だけ GND 記号）"
- moved on the sheet: C100, C101, C102, C103, C104, C105, C106, C107, C108, C109, C110, C111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
