File: kicad/Serrasoid_TRX.kicad_sch (KiCad schematic)
At the start: 327 parts, among them J1 DC 13.8V, J2 I2C, J3 LCD, J4 VOL, J5 ENC, J6 SP, J7 MIC, J8 ANT, J9 TX LED, K1 G5V-2 DC12, Q1 2SC1815, Q10 2SA1015, Q11 2N2222A, Q12 RD06HHF1, Q13 RD16HHF1, Q2 2N3819, Q3 2SC1815, Q4 2SC1815, Q5 2SC1815, Q6 2SC1815, Q7 2N7000, Q8 2SA1015, Q9 2SA1015, T1 BN43-202 2T:5T, U1 74AC74, U10 NJM2594V, U11 AE-Si5351A, U12 74HCU04, U13 ADS1115 module, U14 MC3361, U15 XIAO ESP32C3, U16 MCP6002, U17 LM386N-1, U18 MCP6004, U19 74HCT123, U2 78L05, U20 74AC14, U21 74AC86, U22 74HCU04, U23 74AC14, U3 74AC00, U4 L7808, U5 R-78E5.0-1.0, U6 L7805, U7 MCP6002, U8 LP2950-3.3, U9 AD8307ANZ, X1 10.245MHz, X2 CDBM455C24

Commit message: 終段を IRF510 プッシュプルに変更（RD06HHF1・RD16HHF1 は製造終了）
- ドライバ: RD06HHF1 → IRF510（回路はそのまま、ピンは G-D-S に。アイドル 約 150mA）
- ファイナル: RD16HHF1 → IRF510 × 2 の AB 級プッシュプル。入力トランス BN43-202 1:1（2 次センタータップにバイアス）、
  ゲートストッパー 10Ω・スワンプ 22Ω 1/2W × 2、出力トランス BN43-202 1 次 2 回センタータップ（13.8V 給電）・2 次 3 回（1:2.25）。
  旧ドレインチョーク FT50-43 と結合コンデンサは削除。29MHz・13.8V では出力 約 5W の見込み（仕様を 10W → 約 5W に）
- IRF510 はタブ = ドレインなので、HS1 とケースの放熱器に絶縁シート・絶縁ブッシングで取り付け（部品表に追加）
- センタータップ付き BN43-202 のフットプリント（_SP・_SS、5 ピン）を追加。送信 RF の区画を広げて配置・配線し直し:
  DRC エラー 0・未接続 0・食い違い 0、ERC 0・照合 882 ピン一致
- ケース: ファイナル 2 個の取付ねじ・部品位置・通風スロット、底板 STL・プレビュー（干渉チェック通過）
- スプリアスの図を 5W・プッシュプルの仮定で描き直し（規格線 −13dBm、高調波 最大 −85dBc）
- README・ケースの説明・部品実装図・A3 配置図・回路図 PDF・docx・図・ガーバー・購入用部品表（IRF510・22Ω 1/2W・絶縁キット）、
  回路図論理チェック・基板チェックの追補

Co-Authored-By: Claude Opus 5.5 <noreply@anthropic.com>
Parts:
- removed C125: 0.1u, Capacitor_THT:C_Disc_D5.0mm_W2.5mm_P2.50mm, symbol Device:C
- removed L17: 4.7uH, Inductor_THT:L_Axial_L9.5mm_D4.0mm_P2.54mm_Vertical_Fastron_SMCC, symbol Device:L
- added Q14: IRF510, Package_TO_SOT_THT:TO-220-3_Vertical, symbol Transistor_FET:IRF540N
- added R103: 10k, Resistor_THT:R_Axial_DIN0207_L6.3mm_D2.5mm_P2.54mm_Vertical, symbol Device:R
- added T2: BN43-202 2T(CT):3T, Serrasoid_TRX:Transformer_BN43-202_SP, symbol Device:Transformer_SP_1S
- C104: value 0.01u -> 1000p; footprint Capacitor_THT:C_Disc_D5.0mm_W2.5mm_P2.50mm -> Capacitor_THT:C_Disc_D3.0mm_W1.6mm_P2.50mm
- C106: value 1000p -> 0.1u; footprint Capacitor_THT:C_Disc_D3.0mm_W1.6mm_P2.50mm -> Capacitor_THT:C_Disc_D5.0mm_W2.5mm_P2.50mm
- C110: value 0.1u -> 0.01u
- C111: value 0.01u -> 100p; footprint Capacitor_THT:C_Disc_D5.0mm_W2.5mm_P2.50mm -> Capacitor_THT:C_Disc_D3.0mm_W1.6mm_P2.50mm
- C112: value 220u -> 47p; footprint Capacitor_THT:CP_Radial_D8.0mm_P3.50mm -> Capacitor_THT:C_Disc_D3.0mm_W1.6mm_P2.50mm; symbol Device:C_Polarized -> Device:C
- C113: value 100p -> 0.1u; footprint Capacitor_THT:C_Disc_D3.0mm_W1.6mm_P2.50mm -> Capacitor_THT:C_Disc_D5.0mm_W2.5mm_P2.50mm
- C114: value 47p -> 220u; footprint Capacitor_THT:C_Disc_D3.0mm_W1.6mm_P2.50mm -> Capacitor_THT:CP_Radial_D8.0mm_P3.50mm; symbol Device:C -> Device:C_Polarized
- C115: value 0.1u -> 120p; footprint Capacitor_THT:C_Disc_D5.0mm_W2.5mm_P2.50mm -> Capacitor_THT:C_Disc_D5.0mm_W2.5mm_P5.00mm
- C116: value 120p -> 220p
- C117: value 220p -> 100p; footprint Capacitor_THT:C_Disc_D5.0mm_W2.5mm_P5.00mm -> Capacitor_THT:C_Disc_D3.0mm_W1.6mm_P2.50mm
- C119: value 120p -> 1000p; footprint Capacitor_THT:C_Disc_D5.0mm_W2.5mm_P5.00mm -> Capacitor_THT:C_Disc_D3.0mm_W1.6mm_P2.50mm
- C120: value 100p -> 120p; footprint Capacitor_THT:C_Disc_D3.0mm_W1.6mm_P2.50mm -> Capacitor_THT:C_Disc_D5.0mm_W2.5mm_P5.00mm
- C123: value 1000p -> 0.01u; footprint Capacitor_THT:C_Disc_D3.0mm_W1.6mm_P2.50mm -> Capacitor_THT:C_Disc_D5.0mm_W2.5mm_P2.50mm
- C124: value 0.01u -> 0.1u
- L13: value FT50-43 8T -> T50-6 9T
- L14: value T50-6 9T -> 4.7uH; footprint Serrasoid_TRX:L_T50_2pin_Vertical -> Inductor_THT:L_Axial_L9.5mm_D4.0mm_P2.54mm_Vertical_Fastron_SMCC
- Q12: value RD06HHF1 -> IRF510; symbol Serrasoid_TRX:RD_MOSFET_GSD -> Transistor_FET:IRF540N
- Q13: value RD16HHF1 -> IRF510; symbol Serrasoid_TRX:RD_MOSFET_GSD -> Transistor_FET:IRF540N
- R101: value 47k -> 10k
- R102: value 10k -> 47k
- R89: value 100 -> 1k; footprint Resistor_THT:R_Axial_DIN0414_L11.9mm_D4.5mm_P5.08mm_Vertical -> Resistor_THT:R_Axial_DIN0207_L6.3mm_D2.5mm_P2.54mm_Vertical
- R90: value 100 -> 1M; footprint Resistor_THT:R_Axial_DIN0414_L11.9mm_D4.5mm_P5.08mm_Vertical -> Resistor_THT:R_Axial_DIN0207_L6.3mm_D2.5mm_P2.54mm_Vertical
- R91: value 1k -> 1M
- R92: value 10 -> 3.3k
- R93, R94: value 1M -> 22; footprint Resistor_THT:R_Axial_DIN0207_L6.3mm_D2.5mm_P2.54mm_Vertical -> Resistor_THT:R_Axial_DIN0414_L11.9mm_D4.5mm_P5.08mm_Vertical
- R95: value 3.3k -> 10
- R96: value 910 -> 10
- R97: value 330 -> 910
- R98: value 1k -> 330
- R99: value 10k -> 1k
- T1: value BN43-202 2T:5T -> BN43-202 2T:2T(CT); footprint Serrasoid_TRX:Transformer_BN43-202 -> Serrasoid_TRX:Transformer_BN43-202_SS; symbol Device:Transformer_1P_1S -> Device:Transformer_1P_SS
Connections:
- net +13V8: now also C110.1, C114.1, T2.2 (PM); no longer C111.1, C112.1, L13.1
- net +5VT: now also C113.1; no longer C115.1
- net GND: now also C106.2, C110.2, C123.2, L14.2, Q12.3 (S), Q13.3 (S), R102.2, Q14.3 (S), T2.5 (S2); no longer C104.2, C119.2, Q12.2 (S), Q13.2 (S), R99.2, T1.4 (SB)
- net TX8V: now also R92.1; no longer R95.1
- net at U20.10, U21.4: now also R97.1; no longer R96.1
- net at U21.6: now also R99.1; no longer R98.1
- net at C102.1, L11.1, R87.2: now also C104.1; no longer C105.1
- net at C121.1, K1.8, L16.2: now also C120.1; no longer C119.1
- net at D13.1 (K), R102.1: now also C123.1, R103.1; no longer C124.1, R101.1
- net at U15.2 (D1/A1): now also C124.1, R103.2; no longer R102.2
- net at U21.12, U23.2: now also R98.1; no longer R97.1
- net at C108.1, VR7.2: now also R89.1; no longer R91.1
- net at T1.1 (AA): now also C100.2; no longer C110.2
- net at R100.1, U22.3: now also C119.2; no longer C123.2
- net at R95.2: now also Q13.1 (G); no longer VR7.1
- net at C100.1, L10.2: now also Q12.2 (D); no longer Q12.3 (D)
- net at U22.6, U23.1: now also R91.2; no longer R94.2
- net at C121.2, C122.1, D13.2 (A): now also R101.1; no longer R99.1
- net at U20.11, U22.2: now also R90.2; no longer R93.2
- net at C103.1, L12.1, R88.2: now also C105.1; no longer C106.1
- net at R92.2: now also VR7.1; no longer Q13.1 (G)
- new net: C105.2, R91.1, U22.5
- new net: C111.1, R97.2, U20.3
- new net: R94.1, R96.1, T1.3 (SA)
- new net: C106.1, R89.2, R93.2, R94.2, T1.4 (SC)
- new net: R93.1, R95.1, T1.5 (SB)
- new net: C115.1, L13.1, T2.4 (S1)
- new net: C116.1, L13.2, L15.1
- new net: C112.1, R98.2, U20.9
- new net: C117.1, C119.1, L14.1, R99.2
- new net: C104.2, R90.1, U22.1
- new net: Q14.1 (G), R96.2
- new net: Q13.2 (D), T2.1 (PR1)
- new net: Q14.2 (D), T2.3 (PR2)
Other:
- moved on the sheet: C104, C105, C106, C110, C111, C113, C115, C116, C117, C118, C119, C120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

Commit message: ファイナルを MRF101AN に変更（10W に戻す）
- ファイナル: IRF510 × 2 プッシュプル → MRF101AN（NXP LDMOS、TO-220）1 個。回路は RD16HHF1 のときと同じ単段 AB 級
  （ゲートストッパー 10Ω、スワンプ 100Ω 1/2W × 2、ドレインチョーク FT50-43 8 回、結合 0.1µF、BN43-202 2 回:5 回で 8Ω → 50Ω）。
  ピンは 1 = G・2 = S・3 = D、タブ = ソースで RD16HHF1 と同じなので絶縁不要。アイドル 約 200mA（VGS(th) 1.7〜2.7V）
- ドライバ Q12 は IRF510 のまま（HS1 から絶縁）。入力トランス・ファイナル B・22Ω × 2・センタータップ付きフットプリントを削除
- 基板を作り直し: DRC エラー 0・未接続 0・食い違い 0、ERC 0・照合 875 ピン一致。部品位置は単段のときと同じ
- ケースは取付ねじ 1 本の形に戻した（干渉チェック通過）。スプリアスの図は 10W・単段の仮定に戻した
- README（出力 10W）・ケースの説明・部品実装図・A3 配置図・回路図 PDF・docx・ガーバー・部品表（MRF101AN 568-14751-ND、絶縁キット 1 組）、
  回路図論理チェック・基板チェックの追補

Co-Authored-By: Claude Opus 5.5 <noreply@anthropic.com>
Parts:
- removed Q14: IRF510, Package_TO_SOT_THT:TO-220-3_Vertical, symbol Transistor_FET:IRF540N
- removed R103: 10k, Resistor_THT:R_Axial_DIN0207_L6.3mm_D2.5mm_P2.54mm_Vertical, symbol Device:R
- removed T2: BN43-202 2T(CT):3T, Serrasoid_TRX:Transformer_BN43-202_SP, symbol Device:Transformer_SP_1S
- added C125: 0.1u, Capacitor_THT:C_Disc_D5.0mm_W2.5mm_P2.50mm, symbol Device:C
- added L17: 4.7uH, Inductor_THT:L_Axial_L9.5mm_D4.0mm_P2.54mm_Vertical_Fastron_SMCC, symbol Device:L
- C104: value 1000p -> 0.01u; footprint Capacitor_THT:C_Disc_D3.0mm_W1.6mm_P2.50mm -> Capacitor_THT:C_Disc_D5.0mm_W2.5mm_P2.50mm
- C106: value 0.1u -> 1000p; footprint Capacitor_THT:C_Disc_D5.0mm_W2.5mm_P2.50mm -> Capacitor_THT:C_Disc_D3.0mm_W1.6mm_P2.50mm
- C110: value 0.01u -> 0.1u
- C111: value 100p -> 0.01u; footprint Capacitor_THT:C_Disc_D3.0mm_W1.6mm_P2.50mm -> Capacitor_THT:C_Disc_D5.0mm_W2.5mm_P2.50mm
- C112: value 47p -> 220u; footprint Capacitor_THT:C_Disc_D3.0mm_W1.6mm_P2.50mm -> Capacitor_THT:CP_Radial_D8.0mm_P3.50mm; symbol Device:C -> Device:C_Polarized
- C113: value 0.1u -> 100p; footprint Capacitor_THT:C_Disc_D5.0mm_W2.5mm_P2.50mm -> Capacitor_THT:C_Disc_D3.0mm_W1.6mm_P2.50mm
- C114: value 220u -> 47p; footprint Capacitor_THT:CP_Radial_D8.0mm_P3.50mm -> Capacitor_THT:C_Disc_D3.0mm_W1.6mm_P2.50mm; symbol Device:C_Polarized -> Device:C
- C115: value 120p -> 0.1u; footprint Capacitor_THT:C_Disc_D5.0mm_W2.5mm_P5.00mm -> Capacitor_THT:C_Disc_D5.0mm_W2.5mm_P2.50mm
- C116: value 220p -> 120p
- C117: value 100p -> 220p; footprint Capacitor_THT:C_Disc_D3.0mm_W1.6mm_P2.50mm -> Capacitor_THT:C_Disc_D5.0mm_W2.5mm_P5.00mm
- C119: value 1000p -> 120p; footprint Capacitor_THT:C_Disc_D3.0mm_W1.6mm_P2.50mm -> Capacitor_THT:C_Disc_D5.0mm_W2.5mm_P5.00mm
- C120: value 120p -> 100p; footprint Capacitor_THT:C_Disc_D5.0mm_W2.5mm_P5.00mm -> Capacitor_THT:C_Disc_D3.0mm_W1.6mm_P2.50mm
- C123: value 0.01u -> 1000p; footprint Capacitor_THT:C_Disc_D5.0mm_W2.5mm_P2.50mm -> Capacitor_THT:C_Disc_D3.0mm_W1.6mm_P2.50mm
- C124: value 0.1u -> 0.01u
- L13: value T50-6 9T -> FT50-43 8T
- L14: value 4.7uH -> T50-6 9T; footprint Inductor_THT:L_Axial_L9.5mm_D4.0mm_P2.54mm_Vertical_Fastron_SMCC -> Serrasoid_TRX:L_T50_2pin_Vertical
- Q13: value IRF510 -> MRF101AN; symbol Transistor_FET:IRF540N -> Serrasoid_TRX:RD_MOSFET_GSD
- R101: value 10k -> 47k
- R102: value 47k -> 10k
- R89: value 1k -> 100; footprint Resistor_THT:R_Axial_DIN0207_L6.3mm_D2.5mm_P2.54mm_Vertical -> Resistor_THT:R_Axial_DIN0414_L11.9mm_D4.5mm_P5.08mm_Vertical
- R90: value 1M -> 100; footprint Resistor_THT:R_Axial_DIN0207_L6.3mm_D2.5mm_P2.54mm_Vertical -> Resistor_THT:R_Axial_DIN0414_L11.9mm_D4.5mm_P5.08mm_Vertical
- R91: value 1M -> 1k
- R92: value 3.3k -> 10
- R93, R94: value 22 -> 1M; footprint Resistor_THT:R_Axial_DIN0414_L11.9mm_D4.5mm_P5.08mm_Vertical -> Resistor_THT:R_Axial_DIN0207_L6.3mm_D2.5mm_P2.54mm_Vertical
- R95: value 10 -> 3.3k
- R96: value 10 -> 910
- R97: value 910 -> 330
- R98: value 330 -> 1k
- R99: value 1k -> 10k
- T1: value BN43-202 2T:2T(CT) -> BN43-202 2T:5T; footprint Serrasoid_TRX:Transformer_BN43-202_SS -> Serrasoid_TRX:Transformer_BN43-202; symbol Device:Transformer_1P_SS -> Device:Transformer_1P_1S
Connections:
- net +13V8: now also C111.1, C112.1, L13.1; no longer C110.1, C114.1
- net +5VT: now also C115.1; no longer C113.1
- net GND: now also C104.2, C119.2, Q13.2 (S), R99.2, T1.4 (SB), C125.2, L17.2; no longer C106.2, C110.2, C123.2, L14.2, Q13.3 (S), R102.2
- net TX8V: now also R95.1; no longer R92.1
- net at U20.10, U21.4: now also R96.1; no longer R97.1
- net at U21.6: now also R98.1; no longer R99.1
- net at C102.1, L11.1, R87.2: now also C105.1; no longer C104.1
- net at C121.1, K1.8, L16.2: now also C119.1; no longer C120.1
- net at C103.1, L12.1, R88.2: now also C106.1; no longer C105.1
- net at D13.1 (K), R102.1: now also C124.1, R101.1; no longer C123.1
- net at U22.6, U23.1: now also R94.2; no longer R91.2
- net at C100.2: now also R89.1, R90.1, R91.2, R92.1; no longer T1.1 (AA)
- net at U21.12, U23.2: now also R97.1; no longer R98.1
- net at R100.1, U22.3: now also C123.2; no longer C119.2
- net at C121.2, C122.1, D13.2 (A): now also R99.1; no longer R101.1
- net at R95.2: now also VR7.1; no longer Q13.1 (G)
- net at R92.2: now also Q13.1 (G); no longer VR7.1
- net at C108.1, VR7.2: now also R91.1; no longer R89.1
- net at R96.2: now also C113.1, U20.3
- net at U20.11, U22.2: now also R93.2; no longer R90.2
- net at U15.2 (D1/A1): now also R102.2, C125.1; no longer C124.1
- new net: C105.2, R93.1, U22.1
- new net: C114.1, R97.2, U20.9
- new net: C110.2, T1.1 (AA)
- new net: C116.1, L14.1, T1.3 (SA)
- new net: C120.1, C123.1, L17.1, R98.2
- new net: C110.1, L13.2, Q13.3 (D)
- new net: C117.1, L14.2, L15.1
- new net: C104.1, R89.2, R90.2
- new net: C106.2, R94.1, U22.5
Other:
- moved on the sheet: C104, C105, C106, C110, C111, C113, C115, C116, C117, C118, C119, C120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

Commit message: ファイナルを IRF510 プッシュプルに戻す（MRF101AN は高価なため）
- cfc4ac1（MRF101AN）を取り消し、0b510b6 の IRF510 × 2 プッシュプル（約 5W）に戻した。
  回路・基板・部品表・README などは 0b510b6 と同じ。ERC 0・照合 882 ピン一致、DRC エラー 0・未接続 0・食い違い 0
- 残っていた「10W」の表記を直した: 回路図の題名・docx の副題を「29MHz FM 5W トランシーバ」に、
  ケース前面の刻印を「29MHz FM 5W」に（前面パネル STL を再出力）
- A3 配置図の注記を「DC・ファイナル IRF510・ANT」に

Co-Authored-By: Claude Opus 5.5 <noreply@anthropic.com>
Parts:
- removed C125: 0.1u, Capacitor_THT:C_Disc_D5.0mm_W2.5mm_P2.50mm, symbol Device:C
- removed L17: 4.7uH, Inductor_THT:L_Axial_L9.5mm_D4.0mm_P2.54mm_Vertical_Fastron_SMCC, symbol Device:L
- added Q14: IRF510, Package_TO_SOT_THT:TO-220-3_Vertical, symbol Transistor_FET:IRF540N
- added R103: 10k, Resistor_THT:R_Axial_DIN0207_L6.3mm_D2.5mm_P2.54mm_Vertical, symbol Device:R
- added T2: BN43-202 2T(CT):3T, Serrasoid_TRX:Transformer_BN43-202_SP, symbol Device:Transformer_SP_1S
- C104: value 0.01u -> 1000p; footprint Capacitor_THT:C_Disc_D5.0mm_W2.5mm_P2.50mm -> Capacitor_THT:C_Disc_D3.0mm_W1.6mm_P2.50mm
- C106: value 1000p -> 0.1u; footprint Capacitor_THT:C_Disc_D3.0mm_W1.6mm_P2.50mm -> Capacitor_THT:C_Disc_D5.0mm_W2.5mm_P2.50mm
- C110: value 0.1u -> 0.01u
- C111: value 0.01u -> 100p; footprint Capacitor_THT:C_Disc_D5.0mm_W2.5mm_P2.50mm -> Capacitor_THT:C_Disc_D3.0mm_W1.6mm_P2.50mm
- C112: value 220u -> 47p; footprint Capacitor_THT:CP_Radial_D8.0mm_P3.50mm -> Capacitor_THT:C_Disc_D3.0mm_W1.6mm_P2.50mm; symbol Device:C_Polarized -> Device:C
- C113: value 100p -> 0.1u; footprint Capacitor_THT:C_Disc_D3.0mm_W1.6mm_P2.50mm -> Capacitor_THT:C_Disc_D5.0mm_W2.5mm_P2.50mm
- C114: value 47p -> 220u; footprint Capacitor_THT:C_Disc_D3.0mm_W1.6mm_P2.50mm -> Capacitor_THT:CP_Radial_D8.0mm_P3.50mm; symbol Device:C -> Device:C_Polarized
- C115: value 0.1u -> 120p; footprint Capacitor_THT:C_Disc_D5.0mm_W2.5mm_P2.50mm -> Capacitor_THT:C_Disc_D5.0mm_W2.5mm_P5.00mm
- C116: value 120p -> 220p
- C117: value 220p -> 100p; footprint Capacitor_THT:C_Disc_D5.0mm_W2.5mm_P5.00mm -> Capacitor_THT:C_Disc_D3.0mm_W1.6mm_P2.50mm
- C119: value 120p -> 1000p; footprint Capacitor_THT:C_Disc_D5.0mm_W2.5mm_P5.00mm -> Capacitor_THT:C_Disc_D3.0mm_W1.6mm_P2.50mm
- C120: value 100p -> 120p; footprint Capacitor_THT:C_Disc_D3.0mm_W1.6mm_P2.50mm -> Capacitor_THT:C_Disc_D5.0mm_W2.5mm_P5.00mm
- C123: value 1000p -> 0.01u; footprint Capacitor_THT:C_Disc_D3.0mm_W1.6mm_P2.50mm -> Capacitor_THT:C_Disc_D5.0mm_W2.5mm_P2.50mm
- C124: value 0.01u -> 0.1u
- L13: value FT50-43 8T -> T50-6 9T
- L14: value T50-6 9T -> 4.7uH; footprint Serrasoid_TRX:L_T50_2pin_Vertical -> Inductor_THT:L_Axial_L9.5mm_D4.0mm_P2.54mm_Vertical_Fastron_SMCC
- Q13: value MRF101AN -> IRF510; symbol Serrasoid_TRX:RD_MOSFET_GSD -> Transistor_FET:IRF540N
- R101: value 47k -> 10k
- R102: value 10k -> 47k
- R89: value 100 -> 1k; footprint Resistor_THT:R_Axial_DIN0414_L11.9mm_D4.5mm_P5.08mm_Vertical -> Resistor_THT:R_Axial_DIN0207_L6.3mm_D2.5mm_P2.54mm_Vertical
- R90: value 100 -> 1M; footprint Resistor_THT:R_Axial_DIN0414_L11.9mm_D4.5mm_P5.08mm_Vertical -> Resistor_THT:R_Axial_DIN0207_L6.3mm_D2.5mm_P2.54mm_Vertical
- R91: value 1k -> 1M
- R92: value 10 -> 3.3k
- R93, R94: value 1M -> 22; footprint Resistor_THT:R_Axial_DIN0207_L6.3mm_D2.5mm_P2.54mm_Vertical -> Resistor_THT:R_Axial_DIN0414_L11.9mm_D4.5mm_P5.08mm_Vertical
- R95: value 3.3k -> 10
- R96: value 910 -> 10
- R97: value 330 -> 910
- R98: value 1k -> 330
- R99: value 10k -> 1k
- T1: value BN43-202 2T:5T -> BN43-202 2T:2T(CT); footprint Serrasoid_TRX:Transformer_BN43-202 -> Serrasoid_TRX:Transformer_BN43-202_SS; symbol Device:Transformer_1P_1S -> Device:Transformer_1P_SS
Connections:
- net +13V8: now also C110.1, C114.1, T2.2 (PM); no longer C111.1, C112.1, L13.1
- net +5VT: now also C113.1; no longer C115.1
- net GND: now also C106.2, C110.2, C123.2, L14.2, Q13.3 (S), R102.2, Q14.3 (S), T2.5 (S2); no longer C104.2, C119.2, Q13.2 (S), R99.2, T1.4 (SB)
- net TX8V: now also R92.1; no longer R95.1
- net at U20.10, U21.4: now also R97.1; no longer R96.1
- net at U21.6: now also R99.1; no longer R98.1
- net at C102.1, L11.1, R87.2: now also C104.1; no longer C105.1
- net at C121.1, K1.8, L16.2: now also C120.1; no longer C119.1
- net at D13.1 (K), R102.1: now also C123.1, R103.1; no longer C124.1, R101.1
- net at U15.2 (D1/A1): now also C124.1, R103.2; no longer R102.2
- net at U21.12, U23.2: now also R98.1; no longer R97.1
- net at C108.1, VR7.2: now also R89.1; no longer R91.1
- net at T1.1 (AA): now also C100.2; no longer C110.2
- net at R100.1, U22.3: now also C119.2; no longer C123.2
- net at R95.2: now also Q13.1 (G); no longer VR7.1
- net at U22.6, U23.1: now also R91.2; no longer R94.2
- net at C121.2, C122.1, D13.2 (A): now also R101.1; no longer R99.1
- net at U20.11, U22.2: now also R90.2; no longer R93.2
- net at C103.1, L12.1, R88.2: now also C105.1; no longer C106.1
- net at R92.2: now also VR7.1; no longer Q13.1 (G)
- new net: C105.2, R91.1, U22.5
- new net: C111.1, R97.2, U20.3
- new net: R94.1, R96.1, T1.3 (SA)
- new net: C106.1, R89.2, R93.2, R94.2, T1.4 (SC)
- new net: R93.1, R95.1, T1.5 (SB)
- new net: C115.1, L13.1, T2.4 (S1)
- new net: C116.1, L13.2, L15.1
- new net: C112.1, R98.2, U20.9
- new net: C117.1, C119.1, L14.1, R99.2
- new net: C104.2, R90.1, U22.1
- new net: Q14.1 (G), R96.2
- new net: Q13.2 (D), T2.1 (PR1)
- new net: Q14.2 (D), T2.3 (PR2)
Other:
- title: Serrasoid TRX 29M（セラゾイド変調 29MHz FM 10W トランシーバ） -> Serrasoid TRX 29M（セラゾイド変調 29MHz FM 5W トランシーバ）
- moved on the sheet: C104, C105, C106, C110, C111, C113, C115, C116, C117, C118, C119, C120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
