File: kicad/Serrasoid_TRX.kicad_pcb (KiCad board)
At the start: 4 copper layers, 170 x 140 mm, 310 parts, among them J1 DC 13.8V, J2 I2C, J3 TJC, J4 VOL, J5 ENC, J6 SP, J7 MIC, J8 ANT, J9 TX LED, K1 G5V-2 DC12, Q1 2N3819, Q10 RD16HHF1, Q2 2SC1815, Q3 2SC1815, Q4 2SC1815, Q5 2SC1815, Q6 2N7000, Q7 2SA1015, Q8 2N3866, Q9 RD06HHF1, T1 BN43-202 2T:5T, U1 74AC74, U10 AE-Si5351A, U11 74HCU04, U12 MC3361, U13 XIAO ESP32C3, U14 MCP6002, U15 LM386N-1, U16 MCP6004, U17 74HCT4017, U18 MAX913CPA, U19 74HCT123, U2 78L05, U20 74AC14, U21 74AC86, U22 74HCU04, U23 74AC14, U3 74AC00, U4 L7808, U5 R-78E5.0-1.0, U6 L7805, U7 MCP6002, U8 LP2950-3.3, U9 NJM2594V, X1 10.245MHz, X2 CDBM455C24

Commit message: スケッチを追加（Nextion / TJC 両対応、アナログ S メーター、周波数スキャン）
- firmware/Serrasoid_TRX/Serrasoid_TRX.ino（XIAO ESP32C3、コンパイル確認のみ・実機未確認）
  - Si5351: CLK0 = 送信周波数 × 10 ÷ 16（送信中だけ）、CLK1 = 受信周波数 − 10.7MHz（受信中だけ）
  - PTT: 局発を止める → リレー → 15ms → 変調基準。29.000〜29.700MHz の外では送信しない
  - 操作: ダイヤル = 周波数、押す = メニュー（STEP / SQL / SCAN / EXIT）、長押し = 呼出 29.300MHz
  - スキャン: 10kHz ずつ、スケルチが開いたら止まり、信号が消えて 3 秒で再開
  - S メーターは RSSI がないのでスケルチ用ノイズの減り方から換算（目安、S5 前後で頭打ち）、送信中は出力 W
- firmware/Serrasoid_TRX/nextion/: 背景画像（S メーター＋出力 W の目盛り）、表示の見本、画面データ作成手順
  （Nextion NX4832T035 = Nextion Editor、TJC4832T135 = USART HMI。スケッチは共通。.HMI / .tft は未作成）
- 表示器を Nextion NX4832T035（PSN_TRX と同じ）に、TJC4832T135 も可。J3 の値 TJC → LCD
  （2 番 = XIAO の TX → 表示器の RX（黄））。部品表・購入用部品表・README・ケースの説明を更新
- 回路図 ERC 0・照合 835 ピン一致、基板 DRC エラー 0・未接続 0・食い違い 0

Co-Authored-By: Claude Opus 5.5 <noreply@anthropic.com>
Parts:
- J3: value TJC -> LCD
Changed lines of the file:
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@@
 			)
 		)
-		(property "Value" "TJC"
+		(property "Value" "LCD"
 			(at 0 10 270)
 			(layer "F.Fab")
