File: kicad/Serrasoid_TRX.kicad_pcb (KiCad board)
At the start: 4 copper layers, 170 x 150 mm, 329 parts, among them J1 DC 13.8V, J2 I2C, J3 LCD, J4 VOL, J5 ENC, J6 SP, J7 MIC, J8 ANT, J9 TX LED, K1 G5V-2 DC12, Q1 2SC1815, Q10 RD06HHF1, Q11 RD16HHF1, Q2 2N3819, Q3 2SC1815, Q4 2SC1815, Q5 2SC1815, Q6 2SC1815, Q7 2N7000, Q8 2SA1015, Q9 2N3866, T1 BN43-202 2T:5T, U1 74AC74, U10 NJM2594V, U11 AE-Si5351A, U12 74HCU04, U13 ADS1115 module, U14 MC3361, U15 XIAO ESP32C3, U16 MCP6002, U17 LM386N-1, U18 MCP6004, U19 74HCT4017, U2 78L05, U20 MAX913CPA, U21 74HCT123, U22 74AC14, U23 74AC86, U24 74HCU04, U25 74AC14, U3 74AC00, U4 L7808, U5 R-78E5.0-1.0, U6 L7805, U7 MCP6002, U8 LP2950-3.3, U9 AD8307ANZ, X1 10.245MHz, X2 CDBM455C24

Commit message: クレジットを変更
Co-Authored-By: Claude Opus 5.5 <noreply@anthropic.com>
Other:
- board text added: "Serrasoid TRX 29M Ver 1.2 Designed by JA6FUF/JH1XHX"
- board text removed: "Serrasoid TRX 29M Ver 1.2 Designed by JA6FUF"
Changed lines of the file:
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@@
 		(layer "Edge.Cuts")
 	)
-	(gr_text "Serrasoid TRX 29M  Ver 1.2  Designed by JA6FUF"
+	(gr_text "Serrasoid TRX 29M  Ver 1.2  Designed by JA6FUF/JH1XHX"
 		(at 85 147.55 0)
 		(layer "B.SilkS")
